File: DIN Relay/MCU.brd (EAGLE design)
At the start: 100 x 80 mm, 7 parts, among them X1 GLX-S-88M, X2 GLX-S-88M, X3 GLX-S-88M, X4 GLX-S-88M, X5 GLX-S-88M, X6 GLX-S-88M

Commit message: MCU changes
Parts:
- added C1, C3: (no value), eagle-ltspice:C1206
- added C2: (no value), adafruit:153CLV-0807
- added K1: 691313410004, Wurth_Elektronik_Electromechanic_Terminal_Blocks_Connectors_rev15c:691313410004
- added R1: (no value), eagle-ltspice:R1206
- added U1: MAX487ESA+TCBX, MAX487ESA_TCBX:SOIC127P600X175-8N
Connections:
- new net N$1: U$1.D18, U1.4
- new net N$2: U$1.D19, U1.1
- new net N$3: U$1.D2, U1.2, U1.3
- new net N$4: K1.3, R1.1, U1.6
- new net N$5: K1.2, R1.2, U1.7
- net N$12: now also C1.2, C2.+, C3.2, K1.1, U1.8
- net N$13: now also U$1.D22; no longer U$1.D19
- net N$6: now also C1.1, C2.-, C3.1, K1.4, U1.5
Routing:
- net N$6: track 208.8 -> 353.3 mm, vias 0 -> 11
- net N$12: track 217.7 -> 291.0 mm
- net N$2: track 0.00 -> 59.7 mm
- net N$1: track 0.00 -> 53.8 mm
- net N$3: track 0.00 -> 51.1 mm
- net N$4: track 0.00 -> 25.8 mm
- net N$5: track 0.00 -> 20.9 mm
- net N$13: track 165.6 -> 151.5 mm
