File: DIN Relay/MCU.sch (EAGLE design)
At the start: 7 parts, among them X1 GLX-S-88M, X2 GLX-S-88M, X3 GLX-S-88M, X4 GLX-S-88M, X5 GLX-S-88M, X6 GLX-S-88M

Commit message: MCU changes
Parts:
- added C1, C3: (no value), eagle-ltspice:CC1206
- added C2: (no value), adafruit:CPOL-US153CLV-0807
- added K1: 691313410004, Wurth_Elektronik_Electromechanic_Terminal_Blocks_Connectors_rev15c:691313410004
- added R1: (no value), eagle-ltspice:RR1206
- added U1: MAX487ESA+TCBX, MAX487ESA_TCBX:MAX487ESA+TCBX
Connections:
- new net N$1: U$1.D18, U1.DI
- new net N$2: U$1.D19, U1.RO
- new net N$3: U$1.D2, U1.DE, U1.~RE
- new net N$4: K1.3, R1.1, U1.A
- new net N$5: K1.2, R1.2, U1.B
- net N$12: now also C1.2, C2.+, C3.2, K1.1, U1.VCC
- net N$13: now also U$1.D22; no longer U$1.D19
- net N$6: now also C1.1, C2.-, C3.1, K1.4, U1.GND
