File: dom-inteligentny/temp-sensor/temp-sensor.brd (EAGLE design)
At the start: 44.8 x 43.3 mm, 15 parts, among them Q1 16MHz, U1 ATMEGA328, U2 MAX487ESA+TCBX, X1 TERMINAL-BLOCK-3.5MM-3-PIN-LO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

Commit message: temp sensor changes
Parts:
- added IC1: REG1117, burr-brown:SOT223
- moved C4 6.82 mm to (11.7, 37.1)
- moved U$1 3.78 mm to (26.7, 23.1)
- moved R1 0.90 mm to (20.4, 21.5)
- moved C6 0.68 mm to (24.4, 41.0), turned to 270 degrees
Connections:
- new net N$3: CN2.3, IC1.3
- net GND: now also IC1.1
- net VCC: now also IC1.2; no longer CN2.3
Routing:
- net GND: track 177.9 -> 195.1 mm
- net N$3: track 0.00 -> 7.92 mm
- net VCC: track 149.9 -> 148.7 mm
- net A4: track 16.6 -> 15.7 mm
- net RST: track 32.5 -> 31.8 mm
