File: dom-inteligentny/temp-sensor/temp-sensor.brd (EAGLE design)
At the start: 44.8 x 43.3 mm, 19 parts, among them IC1 REG1117, Q1 16MHz, U1 ATMEGA328, U2 MAX487ESA+TCBX, X2 TERMINAL-BLOCK-3.5MM-4-PIN-LO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

Commit message: fixes
Parts:
- added R4: 120R, eagle-ltspice:R0603
- C1, C2: device adafruit:C1206 -> eagle-ltspice:C0805
Connections:
- net A: now also R4.2
- net B: now also R4.1
Routing:
- net VCC: track 149.4 -> 165.8 mm
- net GND: track 188.0 -> 188.9 mm
- net A: track 5.44 -> 5.95 mm
Changed lines of the file:
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@@
 <?xml version="1.0" encoding="utf-8"?>
 <!DOCTYPE eagle SYSTEM "eagle.dtd">
-<eagle version="9.2.2">
+<eagle version="9.6.2">
 <drawing>
 <settings>
@@
 </autorouter>
 <elements>
-<element name="C1" library="adafruit" package="C1206" value="22pF" x="37.846" y="21.717" smashed="yes">
+<element name="C1" library="eagle-ltspice" library_urn="urn:adsk.eagle:library:217" package="C0805" package3d_urn="urn:adsk.eagle:package:13265/1" value="22pF" x="37.846" y="21.717" smashed="yes">
 <attribute name="NAME" x="33.02" y="21.209" size="1.27" layer="25"/>
-</element>
-<element name="C2" library="adafruit" package="C1206" value="22pF" x="43.053" y="21.717" smashed="yes" rot="R180">
+<attribute name="SPICEMODEL" value="NONE" x="37.846" y="21.717" size="1.778" layer="27" display="off"/>
+<attribute name="SPICEPREFIX" value="C" x="37.846" y="21.717" size="1.778" layer="27" display="off"/>
+</element>
+<element name="C2" library="eagle-ltspice" library_urn="urn:adsk.eagle:library:217" package="C0805" package3d_urn="urn:adsk.eagle:package:13265/1" value="22pF" x="43.053" y="21.717" smashed="yes" rot="R180">
 <attribute name="NAME" x="46.609" y="20.447" size="1.27" layer="25" rot="R180"/>
+<attribute name="SPICEMODEL" value="NONE" x="43.053" y="21.717" size="1.778" layer="27" rot="R180" display="off"/>
+<attribute name="SPICEPREFIX" value="C" x="43.053" y="21.717" size="1.778" layer="27" rot="R180" display="off"/>
 </element>
 <element name="C3" library="adafruit" package="C0805" value="0.1uF" x="24.13" y="17.272" smashed="yes" rot="R180">
@@
 </element>
 <element name="U$1" library="GY-BMP280" package="GY-BMP280" value="GY-BMP280" x="26.67" y="23.114" smashed="yes">
-<attribute name="NAME" x="31.831" y="30.454" size="1.27" layer="25"/>
 <attribute name="VALUE" x="14.272" y="22.46" size="1.27" layer="27" rot="R90"/>
 </element>
@@
 <attribute name="MF" value="Maxim Integrated" x="64.77" y="78.74" size="1.778" layer="27" rot="R90" display="off"/>
 <attribute name="MP" value="MAX487ESA+TCBX" x="64.77" y="78.74" size="1.778" layer="27" rot="R90" display="off"/>
-<attribute name="NAME" x="38.48003125" y="36.168840625" size="2.08325" layer="25" ratio="10" rot="SR90"/>
 <attribute name="PACKAGE" value="SOIC-8 Maxim Integrated" x="64.77" y="78.74" size="1.778" layer="27" rot="R90" display="off"/>
 <attribute name="PRICE" value="None" x="64.77" y="78.74" size="1.778" layer="27" rot="R90" display="off"/>
@@
 <attribute name="SPICEPREFIX" value="R" x="30.0482" y="34.4424" size="1.778" layer="27" rot="R270" display="off"/>
 <attribute name="VALUE" x="27.5082" y="35.7124" size="1.27" layer="27" rot="R270"/>
+</element>
+<element name="R4" library="eagle-ltspice" library_urn="urn:adsk.eagle:library:217" package="R0603" package3d_urn="urn:adsk.eagle:package:13302/1" value="120R" x="33.1724" y="45.1612" smashed="yes">
+<attribute name="NAME" x="35.3822" y="44.6786" size="1.27" layer="25"/>
+<attribute name="SPICEMODEL" value="NONE" x="33.1724" y="45.1612" size="1.778" layer="27" display="off"/>
+<attribute name="SPICEPREFIX" value="R" x="33.1724" y="45.1612" size="1.778" layer="27" display="off"/>
 </element>
 </elements>
@@
 <contactref element="C2" pad="1"/>
 <wire x1="41.9862" y1="17.6276" x2="41.9862" y2="19.2502" width="0.508" layer="1"/>
-<wire x1="41.9862" y1="19.2502" x2="44.453" y2="21.717" width="0.508" layer="1"/>
+<wire x1="41.9862" y1="19.2502" x2="44.003" y2="21.717" width="0.508" layer="1"/>
 <wire x1="41.9862" y1="17.6276" x2="40.2336" y2="15.875" width="0.508" layer="1"/>
 <wire x1="40.2336" y1="15.875" x2="35.052" y2="15.875" width="0.508" layer="1"/>
@@
 <contactref element="C1" pad="1"/>
 <wire x1="37.1602" y1="17.6276" x2="37.1602" y2="21.0028" width="0.508" layer="1"/>
-<wire x1="37.1602" y1="21.0028" x2="36.446" y2="21.717" width="0.508" layer="1"/>
+<wire x1="37.1602" y1="21.0028" x2="36.896" y2="21.717" width="0.508" layer="1"/>
 <wire x1="37.1602" y1="17.6276" x2="32.4104" y2="22.3774" width="0.508" layer="1"/>
 <wire x1="32.4104" y1="22.3774" x2="30.74" y2="22.3774" width="0.508" layer="1"/>
@@
 <wire x1="34.29" y1="40.894" x2="34.925" y2="41.529" width="0.508" layer="1"/>
 <wire x1="26.74" y1="22.3774" x2="26.74" y2="24.073" width="0.508" layer="1"/>
-<wire x1="39.246" y1="21.717" x2="40.386" y2="21.717" width="0.508" layer="1"/>
-<wire x1="40.386" y1="21.717" x2="41.653" y2="21.717" width="0.508" layer="1"/>
+<wire x1="38.796" y1="21.717" x2="40.386" y2="21.717" width="0.508" layer="1"/>
+<wire x1="40.386" y1="21.717" x2="42.103" y2="21.717" width="0.508" layer="1"/>
 <wire x1="40.64" y1="40.767" x2="45.085" y2="36.322" width="0.8128" layer="16"/>
 <wire x1="45.085" y1="29.21" x2="43.688" y2="27.813" width="0.8128" layer="16"/>
@@
 <wire x1="26.9358" y1="35.2162" x2="27.8384" y2="35.2162" width="0.4064" layer="1"/>
 <wire x1="27.54" y1="31.6928" x2="26.5684" y2="32.6644" width="0.4064" layer="1"/>
-<polygon width="0.4064" layer="16">
+<polygon width="0.4064" layer="16" isolate="0.6096">
 <vertex x="3.302" y="37.9984"/>
 <vertex x="7.366" y="44.3484"/>
@@
 <wire x1="28.3464" y1="12.0184" x2="28.3464" y2="9.7282" width="1.27" layer="1"/>
 <wire x1="28.3464" y1="9.7282" x2="27.8892" y2="9.7282" width="1.27" layer="1"/>
-<wire x1="26.797" y1="38.608" x2="29.94" y2="30.9626" width="0" layer="19" extent="1-1"/>
+<wire x1="5.08" y1="21.844" x2="5.1308" y2="21.8948" width="0.508" layer="1"/>
+<wire x1="19.4814" y1="20.041" x2="20.701" y2="20.041" width="0.508" layer="1"/>
+<wire x1="5.1308" y1="21.8948" x2="17.6276" y2="21.8948" width="0.508" layer="1"/>
+<wire x1="17.6276" y1="21.8948" x2="19.4814" y2="20.041" width="0.508" layer="1"/>
 </signal>
 <signal name="RST">
@@
 <contactref element="U2" pad="6"/>
 <contactref element="CN2" pad="1"/>
-<wire x1="33.655" y1="43.1038" x2="33.655" y2="45.847" width="0.508" layer="1"/>
+<wire x1="33.655" y1="43.1038" x2="33.655" y2="44.8056" width="0.508" layer="1"/>
+<wire x1="33.655" y1="44.8056" x2="33.655" y2="45.847" width="0.508" layer="1"/>
 <wire x1="33.655" y1="45.847" x2="31.75" y2="47.752" width="0.508" layer="1"/>
+<contactref element="R4" pad="2"/>
+<wire x1="34.0224" y1="45.1612" x2="33.6668" y2="44.8056" width="0.508" layer="1"/>
+<wire x1="33.6668" y1="44.8056" x2="33.655" y2="44.8056" width="0.508" layer="1"/>
 </signal>
 <signal name="B">
 <contactref element="U2" pad="7"/>
 <contactref element="CN2" pad="2"/>
-<wire x1="32.385" y1="43.1038" x2="32.385" y2="45.085" width="0.508" layer="1"/>
+<wire x1="32.385" y1="43.1038" x2="32.385" y2="43.8912" width="0.508" layer="1"/>
+<wire x1="32.385" y1="43.8912" x2="32.385" y2="45.085" width="0.508" layer="1"/>
 <wire x1="32.385" y1="45.085" x2="31.75" y2="45.72" width="0.508" layer="1"/>
 <wire x1="31.75" y1="45.72" x2="30.48" y2="45.72" width="0.508" layer="1"/>
 <wire x1="30.48" y1="45.72" x2="29.21" y2="46.99" width="0.508" layer="1"/>
 <wire x1="29.21" y1="46.99" x2="29.21" y2="47.752" width="0.508" layer="1"/>
+<contactref element="R4" pad="1"/>
+<wire x1="32.3224" y1="45.1612" x2="32.385" y2="45.0986" width="0.508" layer="1"/>
+<wire x1="32.385" y1="45.0986" x2="32.385" y2="45.085" width="0.508" layer="1"/>
 </signal>
 <signal name="N$3">
