File: dom-inteligentny/temp-sensor/temp-sensor.sch (EAGLE design)
At the start: 15 parts, among them Q1 16MHz, U1 ATMEGA328, U2 MAX487ESA+TCBX, X1 TERMINAL-BLOCK-3.5MM-3-PIN-LO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

Commit message: temp sensor changes
Parts:
- added IC1: REG1117, burr-brown:REG1117
Connections:
- new net N$3: CN2.3, IC1.VIN
- net GND: now also IC1.GND
- net VCC: now also IC1.VOUT; no longer CN2.3
Changed lines of the file:
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@@
 <part name="GND5" library="SparkFun" deviceset="GND" device=""/>
 <part name="P+7" library="SparkFun" deviceset="VCC" device=""/>
+<part name="IC1" library="burr-brown" library_urn="urn:adsk.eagle:library:111" deviceset="REG1117" device="" package3d_urn="urn:adsk.eagle:package:4940/1"/>
 </parts>
 <sheets>
@@
 <instance part="P+7" gate="1" x="114.3" y="210.82" smashed="yes">
 <attribute name="VALUE" x="113.284" y="214.376" size="1.778" layer="96"/>
+</instance>
+<instance part="IC1" gate="G$1" x="96.52" y="157.48" smashed="yes">
+<attribute name="NAME" x="88.9" y="163.195" size="1.778" layer="95" ratio="10"/>
+<attribute name="VALUE" x="91.44" y="160.02" size="1.778" layer="96" ratio="10"/>
 </instance>
 </instances>
@@
 <segment>
 <pinref part="CN2" gate="G$1" pin="5"/>
-<wire x1="63.5" y1="134.62" x2="71.12" y2="134.62" width="0.1524" layer="91"/>
+<wire x1="63.5" y1="134.62" x2="68.58" y2="134.62" width="0.1524" layer="91"/>
 <label x="71.12" y="134.62" size="1.778" layer="95" xref="yes"/>
+<pinref part="IC1" gate="G$1" pin="GND"/>
+<wire x1="68.58" y1="134.62" x2="71.12" y2="134.62" width="0.1524" layer="91"/>
+<wire x1="96.52" y1="144.78" x2="68.58" y2="144.78" width="0.1524" layer="91"/>
+<wire x1="68.58" y1="144.78" x2="68.58" y2="134.62" width="0.1524" layer="91"/>
+<junction x="68.58" y="134.62"/>
 </segment>
 <segment>
@@
 <wire x1="203.2" y1="78.74" x2="193.04" y2="78.74" width="0.1524" layer="91"/>
 <label x="193.04" y="78.74" size="1.778" layer="95" rot="R180" xref="yes"/>
-</segment>
-<segment>
-<pinref part="CN2" gate="G$1" pin="3"/>
-<wire x1="63.5" y1="129.54" x2="71.12" y2="129.54" width="0.1524" layer="91"/>
-<label x="71.12" y="129.54" size="1.778" layer="95" xref="yes"/>
 </segment>
 <segment>
@@
 <pinref part="P+7" gate="1" pin="VCC"/>
 </segment>
+<segment>
+<pinref part="IC1" gate="G$1" pin="VOUT"/>
+<wire x1="109.22" y1="157.48" x2="114.3" y2="157.48" width="0.1524" layer="91"/>
+<label x="114.3" y="157.48" size="1.778" layer="95" xref="yes"/>
+</segment>
 </net>
 <net name="RST" class="0">
@@
 </segment>
 </net>
+<net name="N$3" class="0">
+<segment>
+<pinref part="IC1" gate="G$1" pin="VIN"/>
+<wire x1="83.82" y1="157.48" x2="66.04" y2="157.48" width="0.1524" layer="91"/>
+<wire x1="66.04" y1="157.48" x2="66.04" y2="129.54" width="0.1524" layer="91"/>
+<pinref part="CN2" gate="G$1" pin="3"/>
+<wire x1="66.04" y1="129.54" x2="63.5" y2="129.54" width="0.1524" layer="91"/>
+</segment>
+</net>
