File: dom-inteligentny/temp-sensor/temp-sensor.sch (EAGLE design)
At the start: 15 parts, among them Q1 16MHz, U1 ATMEGA328, U2 MAX487ESA+TCBX, X1 TERMINAL-BLOCK-3.5MM-3-PIN-LO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

Commit message: new files
Parts:
- added CN1: (no value), con-hdrs40:HDR-1X5-SIP-100
- added CN3: (no value), con-hdrs40:HDR-1X4-SIP-100
Connections:
- net A0: now also CN3.1
- net A1: now also CN3.2
- net A2: now also CN3.3
- net A3: now also CN3.4
- net D7: now also CN1.5
- net D8: now also CN1.3
- net D9: now also CN1.2
- net GND: now also CN1.4
- net VCC: now also CN1.1
Changed lines of the file:
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@@
 <part name="GND5" library="SparkFun" deviceset="GND" device=""/>
 <part name="P+7" library="SparkFun" deviceset="VCC" device=""/>
+<part name="CN1" library="con-hdrs40" deviceset="HDR-1X5" device="-SIP-100"/>
+<part name="CN3" library="con-hdrs40" deviceset="HDR-1X4" device="-SIP-100"/>
 </parts>
 <sheets>
@@
 <attribute name="VALUE" x="113.284" y="214.376" size="1.778" layer="96"/>
 </instance>
+<instance part="CN1" gate="G$1" x="317.5" y="167.64" smashed="yes">
+<attribute name="NAME" x="315.595" y="177.8" size="1.778" layer="95"/>
+<attribute name="VALUE" x="315.595" y="155.8925" size="1.778" layer="96"/>
+</instance>
+<instance part="CN3" gate="G$1" x="317.5" y="149.86" smashed="yes">
+<attribute name="NAME" x="315.595" y="154.94" size="1.778" layer="95"/>
+<attribute name="VALUE" x="315.595" y="140.6525" size="1.778" layer="96"/>
+</instance>
 </instances>
 <busses>
@@
 <label x="248.92" y="187.96" size="1.778" layer="95" xref="yes"/>
 </segment>
+<segment>
+<pinref part="CN3" gate="G$1" pin="1"/>
+<wire x1="312.42" y1="152.4" x2="307.34" y2="152.4" width="0.1524" layer="91"/>
+<label x="307.34" y="152.4" size="1.778" layer="95" rot="R180" xref="yes"/>
+</segment>
 </net>
 <net name="A1" class="0">
@@
 <label x="259.08" y="185.42" size="1.778" layer="95" xref="yes"/>
 </segment>
+<segment>
+<pinref part="CN3" gate="G$1" pin="2"/>
+<wire x1="312.42" y1="149.86" x2="299.72" y2="149.86" width="0.1524" layer="91"/>
+<label x="299.72" y="149.86" size="1.778" layer="95" rot="R180" xref="yes"/>
+</segment>
 </net>
 <net name="A2" class="0">
@@
 <label x="248.92" y="182.88" size="1.778" layer="95" xref="yes"/>
 </segment>
+<segment>
+<pinref part="CN3" gate="G$1" pin="3"/>
+<wire x1="312.42" y1="147.32" x2="307.34" y2="147.32" width="0.1524" layer="91"/>
+<label x="307.34" y="147.32" size="1.778" layer="95" rot="R180" xref="yes"/>
+</segment>
 </net>
 <net name="A3" class="0">
@@
 <wire x1="238.76" y1="180.34" x2="259.08" y2="180.34" width="0.1524" layer="91"/>
 <label x="259.08" y="180.34" size="1.778" layer="95" xref="yes"/>
+</segment>
+<segment>
+<pinref part="CN3" gate="G$1" pin="4"/>
+<wire x1="312.42" y1="144.78" x2="299.72" y2="144.78" width="0.1524" layer="91"/>
+<label x="299.72" y="144.78" size="1.778" layer="95" rot="R180" xref="yes"/>
 </segment>
 </net>
@@
 <label x="259.08" y="147.32" size="1.778" layer="95" xref="yes"/>
 </segment>
+<segment>
+<pinref part="CN1" gate="G$1" pin="5"/>
+<wire x1="312.42" y1="162.56" x2="307.34" y2="162.56" width="0.1524" layer="91"/>
+<label x="307.34" y="162.56" size="1.778" layer="95" rot="R180" xref="yes"/>
+</segment>
 </net>
 <net name="D8" class="0">
@@
 <label x="248.92" y="142.24" size="1.778" layer="95" xref="yes"/>
 </segment>
+<segment>
+<pinref part="CN1" gate="G$1" pin="3"/>
+<wire x1="312.42" y1="167.64" x2="307.34" y2="167.64" width="0.1524" layer="91"/>
+<label x="307.34" y="167.64" size="1.778" layer="95" rot="R180" xref="yes"/>
+</segment>
 </net>
 <net name="D9" class="0">
@@
 <wire x1="238.76" y1="139.7" x2="259.08" y2="139.7" width="0.1524" layer="91"/>
 <label x="259.08" y="139.7" size="1.778" layer="95" xref="yes"/>
+</segment>
+<segment>
+<pinref part="CN1" gate="G$1" pin="2"/>
+<wire x1="312.42" y1="170.18" x2="299.72" y2="170.18" width="0.1524" layer="91"/>
+<label x="299.72" y="170.18" size="1.778" layer="95" rot="R180" xref="yes"/>
 </segment>
 </net>
@@
 <wire x1="114.3" y1="198.12" x2="114.3" y2="193.04" width="0.1524" layer="91"/>
 <pinref part="GND5" gate="1" pin="GND"/>
+</segment>
+<segment>
+<pinref part="CN1" gate="G$1" pin="4"/>
+<wire x1="312.42" y1="165.1" x2="299.72" y2="165.1" width="0.1524" layer="91"/>
+<label x="299.72" y="165.1" size="1.778" layer="95" rot="R180" xref="yes"/>
 </segment>
 </net>
@@
 <pinref part="P+7" gate="1" pin="VCC"/>
 </segment>
-</net>
+<segment>
+<pinref part="CN1" gate="G$1" pin="1"/>
+<wire x1="312.42" y1="172.72" x2="307.34" y2="172.72" width="0.1524" layer="91"/>
+<label x="307.34" y="172.72" size="1.778" layer="95" rot="R180" xref="yes"/>
+</segment>
+</net>
