File: dom-inteligentny/temp-sensor/temp-sensor.sch (EAGLE design)
At the start: 18 parts, among them IC1 REG1117, Q1 16MHz, U1 ATMEGA328, U2 MAX487ESA+TCBX, X1 TERMINAL-BLOCK-3.5MM-3-PIN-LO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

Commit message: Temp sensor, NTC
Parts:
- removed X1: TERMINAL-BLOCK-3.5MM-3-PIN-LONG-PAD, Rembrandt Electronics - Terminal Block 3-5mm v1-0:TERMINAL-BLOCK-3.5MM-3-PIN-LONG-PAD
- added R2: (no value), eagle-ltspice:RR1206
- added X2: TERMINAL-BLOCK-3.5MM-4-PIN-LONG-PAD, Rembrandt Electronics - Terminal Block 3-5mm v1-0:TERMINAL-BLOCK-3.5MM-4-PIN-LONG-PAD
Connections:
- net A6: now also R2.2, X2-1.K
- net D5: now also X2-4.K; no longer X1-3.K
- net GND: now also R2.1, X2-2.K; no longer X1-1.K
- net VCC: now also X2-3.K; no longer X1-2.K
Changed lines of the file:
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@@
 <part name="GND7" library="supply1" library_urn="urn:adsk.eagle:library:371" deviceset="GND" device=""/>
 <part name="P+5" library="supply1" library_urn="urn:adsk.eagle:library:371" deviceset="VCC" device=""/>
-<part name="X1" library="Rembrandt Electronics - Terminal Block 3-5mm v1-0" deviceset="TERMINAL-BLOCK-3.5MM-3-PIN" device="-LONG-PAD"/>
 <part name="C4" library="rcl" library_urn="urn:adsk.eagle:library:334" deviceset="CPOL-EU" device="SANYO_SMD_C6" package3d_urn="urn:adsk.eagle:package:23465/1"/>
 <part name="GND8" library="supply1" library_urn="urn:adsk.eagle:library:371" deviceset="GND" device=""/>
@@
 <part name="CN1" library="con-hdrs40" deviceset="HDR-1X5" device="-SIP-100"/>
 <part name="CN3" library="con-hdrs40" deviceset="HDR-1X4" device="-SIP-100"/>
+<part name="X2" library="Rembrandt Electronics - Terminal Block 3-5mm v1-0" deviceset="TERMINAL-BLOCK-3.5MM-4-PIN" device="-LONG-PAD"/>
+<part name="R2" library="eagle-ltspice" library_urn="urn:adsk.eagle:library:217" deviceset="R" device="R1206" package3d_urn="urn:adsk.eagle:package:13301/1"/>
 </parts>
 <sheets>
@@
 <attribute name="VALUE" x="231.14" y="114.3" size="1.778" layer="96" rot="R90"/>
 </instance>
-<instance part="X1" gate="-1" x="284.48" y="106.68" smashed="yes">
-<attribute name="NAME" x="285.75" y="105.791" size="1.778" layer="95"/>
-<attribute name="VALUE" x="298.45" y="105.791" size="1.778" layer="96"/>
-</instance>
-<instance part="X1" gate="-2" x="284.48" y="99.06" smashed="yes">
-<attribute name="NAME" x="285.75" y="98.171" size="1.778" layer="95"/>
-<attribute name="VALUE" x="298.45" y="98.171" size="1.778" layer="96"/>
-</instance>
-<instance part="X1" gate="-3" x="284.48" y="91.44" smashed="yes">
-<attribute name="NAME" x="285.75" y="90.551" size="1.778" layer="95"/>
-<attribute name="VALUE" x="298.45" y="90.551" size="1.778" layer="96"/>
-</instance>
 <instance part="C4" gate="G$1" x="83.82" y="203.2" smashed="yes">
 <attribute name="NAME" x="84.963" y="203.6826" size="1.778" layer="95"/>
@@
 <attribute name="NAME" x="88.9" y="163.195" size="1.778" layer="95" ratio="10"/>
 <attribute name="VALUE" x="91.44" y="160.02" size="1.778" layer="96" ratio="10"/>
-</instance><instance part="CN1" gate="G$1" x="317.5" y="167.64" smashed="yes">
+</instance>
+<instance part="CN1" gate="G$1" x="317.5" y="167.64" smashed="yes">
 <attribute name="NAME" x="315.595" y="177.8" size="1.778" layer="95"/>
 <attribute name="VALUE" x="315.595" y="155.8925" size="1.778" layer="96"/>
@@
 <attribute name="NAME" x="315.595" y="154.94" size="1.778" layer="95"/>
 <attribute name="VALUE" x="315.595" y="140.6525" size="1.778" layer="96"/>
+</instance>
+<instance part="X2" gate="-1" x="284.48" y="114.3" smashed="yes">
+<attribute name="NAME" x="285.75" y="113.411" size="1.778" layer="95"/>
+</instance>
+<instance part="X2" gate="-2" x="284.48" y="106.68" smashed="yes">
+<attribute name="NAME" x="285.75" y="105.791" size="1.778" layer="95"/>
+</instance>
+<instance part="X2" gate="-3" x="284.48" y="99.06" smashed="yes">
+<attribute name="NAME" x="285.75" y="98.171" size="1.778" layer="95"/>
+</instance>
+<instance part="X2" gate="-4" x="284.48" y="91.44" smashed="yes">
+<attribute name="NAME" x="285.75" y="90.551" size="1.778" layer="95"/>
+</instance>
+<instance part="R2" gate="G$1" x="269.24" y="111.76" smashed="yes" rot="R90">
+<attribute name="NAME" x="267.7414" y="107.95" size="1.778" layer="95" rot="R90"/>
+<attribute name="VALUE" x="272.542" y="107.95" size="1.778" layer="96" rot="R90"/>
 </instance>
 </instances>
@@
 <wire x1="238.76" y1="172.72" x2="248.92" y2="172.72" width="0.1524" layer="91"/>
 <label x="248.92" y="172.72" size="1.778" layer="95" xref="yes"/>
+</segment>
+<segment>
+<pinref part="X2" gate="-1" pin="K"/>
+<wire x1="281.94" y1="114.3" x2="276.86" y2="114.3" width="0.1524" layer="91"/>
+<wire x1="276.86" y1="114.3" x2="276.86" y2="116.84" width="0.1524" layer="91"/>
+<pinref part="R2" gate="G$1" pin="2"/>
+<wire x1="276.86" y1="116.84" x2="269.24" y2="116.84" width="0.1524" layer="91"/>
+<wire x1="269.24" y1="116.84" x2="261.62" y2="116.84" width="0.1524" layer="91"/>
+<junction x="269.24" y="116.84"/>
+<label x="261.62" y="116.84" size="1.778" layer="95" rot="R180" xref="yes"/>
 </segment>
 </net>
@@
 </segment>
 <segment>
-<pinref part="X1" gate="-3" pin="K"/>
 <wire x1="281.94" y1="91.44" x2="279.4" y2="91.44" width="0.1524" layer="91"/>
 <label x="276.86" y="91.44" size="1.778" layer="95" rot="R180" xref="yes"/>
@@
 <wire x1="279.4" y1="91.44" x2="276.86" y2="91.44" width="0.1524" layer="91"/>
 <junction x="279.4" y="91.44"/>
+<pinref part="X2" gate="-4" pin="K"/>
 </segment>
 </net>
@@
 <junction x="248.92" y="104.14"/>
 <wire x1="266.7" y1="104.14" x2="266.7" y2="106.68" width="0.1524" layer="91"/>
-<pinref part="X1" gate="-1" pin="K"/>
-<wire x1="266.7" y1="106.68" x2="281.94" y2="106.68" width="0.1524" layer="91"/>
+<wire x1="266.7" y1="106.68" x2="269.24" y2="106.68" width="0.1524" layer="91"/>
+<pinref part="X2" gate="-2" pin="K"/>
+<pinref part="R2" gate="G$1" pin="1"/>
+<wire x1="269.24" y1="106.68" x2="281.94" y2="106.68" width="0.1524" layer="91"/>
+<junction x="269.24" y="106.68"/>
 </segment>
 <segment>
@@
 <wire x1="279.4" y1="81.28" x2="261.62" y2="81.28" width="0.1524" layer="91"/>
 <wire x1="261.62" y1="81.28" x2="261.62" y2="99.06" width="0.1524" layer="91"/>
-<pinref part="X1" gate="-2" pin="K"/>
 <wire x1="261.62" y1="99.06" x2="261.62" y2="106.68" width="0.1524" layer="91"/>
 <wire x1="281.94" y1="99.06" x2="261.62" y2="99.06" width="0.1524" layer="91"/>
 <junction x="261.62" y="99.06"/>
+<pinref part="X2" gate="-3" pin="K"/>
 </segment>
 <segment>
@@
 <wire x1="109.22" y1="157.48" x2="114.3" y2="157.48" width="0.1524" layer="91"/>
 <label x="114.3" y="157.48" size="1.778" layer="95" xref="yes"/>
-</segment><segment>
+</segment>
+<segment>
 <pinref part="CN1" gate="G$1" pin="1"/>
 <wire x1="312.42" y1="172.72" x2="307.34" y2="172.72" width="0.1524" layer="91"/>
 <label x="307.34" y="172.72" size="1.778" layer="95" rot="R180" xref="yes"/>
-</segment></net>
+</segment>
+</net>
 <net name="RST" class="0">
 <segment>

Commit message: fixes
Parts:
- added R4: 120R, eagle-ltspice:RR0603
- C1, C2: device adafruit:C-USC1206 -> eagle-ltspice:C
Connections:
- net A: now also R4.2
- net B: now also R4.1
Changed lines of the file:
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@@
 <?xml version="1.0" encoding="utf-8"?>
 <!DOCTYPE eagle SYSTEM "eagle.dtd">
-<eagle version="9.2.2">
+<eagle version="9.6.2">
 <drawing>
 <settings>
@@
 <part name="U1" library="thecustomgeek" deviceset="ATMEGA328" device=""/>
 <part name="Q1" library="crystal" deviceset="CRYTAL" device="HC49S" value="16MHz"/>
-<part name="C1" library="adafruit" deviceset="C-US" device="C1206" value="22pF"/>
-<part name="C2" library="adafruit" deviceset="C-US" device="C1206" value="22pF"/>
+<part name="C1" library="eagle-ltspice" library_urn="urn:adsk.eagle:library:217" deviceset="C" device="" package3d_urn="urn:adsk.eagle:package:13265/1" value="22pF"/>
+<part name="C2" library="eagle-ltspice" library_urn="urn:adsk.eagle:library:217" deviceset="C" device="" package3d_urn="urn:adsk.eagle:package:13265/1" value="22pF"/>
 <part name="C3" library="adafruit" deviceset="C-US" device="C0805" value="0.1uF"/>
 <part name="R1" library="adafruit" deviceset="R-US_" device="R1206" value="10K"/>
@@
 <part name="X2" library="Rembrandt Electronics - Terminal Block 3-5mm v1-0" deviceset="TERMINAL-BLOCK-3.5MM-4-PIN" device="-LONG-PAD"/>
 <part name="R2" library="eagle-ltspice" library_urn="urn:adsk.eagle:library:217" deviceset="R" device="R1206" package3d_urn="urn:adsk.eagle:package:13301/1"/>
+<part name="R4" library="eagle-ltspice" library_urn="urn:adsk.eagle:library:217" deviceset="R" device="R0603" package3d_urn="urn:adsk.eagle:package:13302/1" value="120R"/>
 </parts>
 <sheets>
@@
 <attribute name="NAME" x="267.7414" y="107.95" size="1.778" layer="95" rot="R90"/>
 <attribute name="VALUE" x="272.542" y="107.95" size="1.778" layer="96" rot="R90"/>
+</instance>
+<instance part="R4" gate="G$1" x="160.02" y="101.6" smashed="yes" rot="R90">
+<attribute name="NAME" x="158.5214" y="97.79" size="1.778" layer="95" rot="R90"/>
+<attribute name="VALUE" x="163.322" y="97.79" size="1.778" layer="96" rot="R90"/>
 </instance>
 </instances>
@@
 <segment>
 <pinref part="U2" gate="A" pin="A"/>
-<wire x1="154.94" y1="106.68" x2="162.56" y2="106.68" width="0.1524" layer="91"/>
+<wire x1="154.94" y1="106.68" x2="160.02" y2="106.68" width="0.1524" layer="91"/>
 <label x="162.56" y="106.68" size="1.778" layer="95" xref="yes"/>
+<pinref part="R4" gate="G$1" pin="2"/>
+<wire x1="160.02" y1="106.68" x2="162.56" y2="106.68" width="0.1524" layer="91"/>
+<junction x="160.02" y="106.68"/>
 </segment>
 <segment>
@@
 <pinref part="U2" gate="A" pin="B"/>
 <label x="170.18" y="104.14" size="1.778" layer="95" xref="yes"/>
-<wire x1="154.94" y1="104.14" x2="170.18" y2="104.14" width="0.1524" layer="91"/>
-</segment>
-<segment>
+<wire x1="154.94" y1="104.14" x2="165.1" y2="104.14" width="0.1524" layer="91"/>
+<pinref part="R4" gate="G$1" pin="1"/>
+<wire x1="165.1" y1="104.14" x2="170.18" y2="104.14" width="0.1524" layer="91"/>
+<wire x1="160.02" y1="96.52" x2="165.1" y2="96.52" width="0.1524" layer="91"/>
+<wire x1="165.1" y1="96.52" x2="165.1" y2="104.14" width="0.1524" layer="91"/>
+<junction x="165.1" y="104.14"/>
+</segment>
+<segment>
