File: dom-inteligentny/DC/dc.brd (EAGLE design)
At the start: 64 x 88 mm, 8 parts, among them K1 AC, K2 +, K3 -

Commit message: new files
Parts:
- moved C2 4.07 mm to (12.7, 58.4)
- moved K1 1.39 mm to (31.8, 10.0)
- moved K3 1.26 mm to (19.8, 77.9)
- moved K2 1.25 mm to (43.6, 77.9)
- moved C1 1.00 mm to (18.9, 24.2)
Routing:
- net N$6: track 58.0 -> 64.2 mm
- net N$4: track 55.5 -> 56.2 mm
- net N$5: track 65.9 -> 66.6 mm
Other:
- board size 64 x 88 mm -> 64 x 84 mm
- board text added: "Falcon IoT PSU v1.0 weblogic.pl"
