File: dom-inteligentny/MCU/MCU.brd (EAGLE design)
At the start: 100 x 80 mm, 13 parts, among them K1 691313410004, U1 MAX487ESA+TCBX, X1 GLX-S-88M, X2 GLX-S-88M, X3 GLX-S-88M, X4 GLX-S-88M, X5 GLX-S-88M, X6 GLX-S-88M

Commit message: new files
Parts:
- added R2: 4,7k, eagle-ltspice:R1206
Connections:
- net N$6 renamed GND
- removed net N$12: C1.2, C2.+, C3.2, K1.1, U$1.+5V.2, U1.8, X1.7, X1.8, X2.7, X2.8, X3.7, X3.8, X4.7, X4.8, X5.7, X5.8, X6.7, X6.8
- removed net N$13: U$1.D22, X1.2, X2.2, X3.2, X4.2, X5.2, X6.2
- new net INT: R2.2, U$1.D3, X1.2, X2.2, X3.2, X4.2, X5.2, X6.2
- new net VDD: C1.2, C2.+, C3.2, K1.1, R2.1, U$1.+5V.1, U$1.+5V.2, U1.8, X1.7, X1.8, X2.7, X2.8, X3.7, X3.8, X4.7, X4.8, X5.7, X5.8, X6.7, X6.8
Routing:
- net VDD: track 0.00 -> 298.3 mm
- net N$12: track 291.0 -> 0.00 mm
- net INT: track 0.00 -> 178.3 mm
- net N$13: track 151.5 -> 0.00 mm
- net GND: track 353.3 -> 360.5 mm
Other:
- board text added: "Falcon IoT MCU v1.1 weblogic.pl"
Changed lines of the file:
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@@
 <?xml version="1.0" encoding="utf-8"?>
 <!DOCTYPE eagle SYSTEM "eagle.dtd">
-<eagle version="9.2.2">
+<eagle version="9.6.2">
 <drawing>
 <settings>
@@
 <setting verticaltext="up"/>
 </settings>
-<grid distance="10" unitdist="mil" unit="mil" style="lines" multiple="1" display="no" altdistance="5" altunitdist="mil" altunit="mil"/>
+<grid distance="10" unitdist="mil" unit="mil" style="lines" multiple="1" display="no" altdistance="5" altunitdist="mil" altunit="mm"/>
 <layers>
 <layer number="1" name="Top" color="4" fill="1" visible="yes" active="yes"/>
@@
 <layer number="43" name="vRestrict" color="2" fill="10" visible="yes" active="yes"/>
 <layer number="44" name="Drills" color="7" fill="1" visible="no" active="yes"/>
-<layer number="45" name="Holes" color="7" fill="1" visible="no" active="yes"/>
+<layer number="45" name="Holes" color="7" fill="1" visible="yes" active="yes"/>
 <layer number="46" name="Milling" color="3" fill="1" visible="no" active="yes"/>
 <layer number="47" name="Measures" color="7" fill="1" visible="no" active="yes"/>
@@
 <wire x1="100" y1="80" x2="0" y2="80" width="0" layer="20"/>
 <wire x1="0" y1="80" x2="0" y2="0" width="0" layer="20"/>
+<hole x="7" y="15" drill="5"/>
+<hole x="7" y="65" drill="5"/>
+<hole x="93" y="65" drill="5"/>
+<hole x="93" y="15" drill="5"/>
+<text x="71.12" y="37.338" size="1.778" layer="16" rot="MR0">Falcon IoT
+MCU v1.1
+weblogic.pl</text>
 </plain>
 <attributes>
@@
 <attribute name="VALUE" x="12.954" y="72.39" size="1.27" layer="27" rot="R270"/>
 </element>
+<element name="R2" library="eagle-ltspice" library_urn="urn:adsk.eagle:library:217" package="R1206" package3d_urn="urn:adsk.eagle:package:13301/1" value="4,7k" x="31.496" y="18.034" smashed="yes">
+<attribute name="NAME" x="30.226" y="19.304" size="1.27" layer="25"/>
+<attribute name="SPICEMODEL" value="NONE" x="31.496" y="18.034" size="1.778" layer="27" display="off"/>
+<attribute name="SPICEPREFIX" value="R" x="31.496" y="18.034" size="1.778" layer="27" display="off"/>
+<attribute name="VALUE" x="30.226" y="15.494" size="1.27" layer="27"/>
+</element>
 </elements>
 <signals>
-<signal name="N$6">
+<signal name="GND">
 <contactref element="X6" pad="1"/>
 <contactref element="X6" pad="3"/>
@@
 <via x="6.35" y="22.86" extent="1-16" drill="0.35"/>
 <via x="6.35" y="24.13" extent="1-16" drill="0.35"/>
-<wire x1="5.078" y1="34.036" x2="5.078" y2="65.022" width="1.27" layer="1"/>
-<wire x1="5.078" y1="65.022" x2="12.954" y2="72.898" width="1.27" layer="1"/>
-<wire x1="12.954" y1="72.898" x2="41.656" y2="72.898" width="1.27" layer="1"/>
 <wire x1="44.45" y1="70.104" x2="44.45" y2="69.088" width="1.27" layer="1"/>
 <wire x1="41.656" y1="72.898" x2="44.45" y2="70.104" width="1.27" layer="1"/>
 <contactref element="C3" pad="1"/>
-<wire x1="15.494" y1="72.52" x2="14.986" y2="8.0587" width="0" layer="19" extent="1-16"/>
-</signal>
-<signal name="N$12">
+<wire x1="5.078" y1="34.036" x2="5.078" y2="55.882" width="1.27" layer="1"/>
+<wire x1="5.078" y1="55.882" x2="2.54" y2="58.42" width="1.27" layer="1"/>
+<wire x1="2.54" y1="58.42" x2="2.54" y2="70.612" width="1.27" layer="1"/>
+<wire x1="2.54" y1="70.612" x2="4.826" y2="72.898" width="1.27" layer="1"/>
+<wire x1="4.826" y1="72.898" x2="15.494" y2="72.898" width="1.27" layer="1"/>
+<wire x1="15.494" y1="72.898" x2="41.656" y2="72.898" width="1.27" layer="1"/>
+<wire x1="15.494" y1="72.52" x2="15.494" y2="72.898" width="0.508" layer="1"/>
+</signal>
+<signal name="VDD">
 <contactref element="X6" pad="7"/>
 <contactref element="X6" pad="8"/>
@@
 <wire x1="11.178" y1="34.036" x2="11.178" y2="63.246" width="1.27" layer="1"/>
 <wire x1="11.178" y1="63.246" x2="11.178" y2="65.534" width="1.27" layer="1"/>
-<wire x1="14.732" y1="69.088" x2="21.59" y2="69.088" width="1.27" layer="1"/>
+<wire x1="14.732" y1="69.088" x2="15.494" y2="69.088" width="1.27" layer="1"/>
+<wire x1="15.494" y1="69.088" x2="21.59" y2="69.088" width="1.27" layer="1"/>
 <wire x1="11.178" y1="65.534" x2="14.732" y2="69.088" width="1.27" layer="1"/>
 <wire x1="14.351" y1="63.1698" x2="14.2748" y2="63.246" width="0.6096" layer="1"/>
 <wire x1="14.2748" y1="63.246" x2="11.178" y2="63.246" width="0.6096" layer="1"/>
 <contactref element="C3" pad="2"/>
-<wire x1="15.494" y1="69.72" x2="16.75" y2="9.67" width="0" layer="19" extent="1-1"/>
-</signal>
-<signal name="N$13">
+<wire x1="15.494" y1="69.72" x2="15.494" y2="69.088" width="0.508" layer="1"/>
+<contactref element="U$1" pad="+5V.1"/>
+<contactref element="R2" pad="1"/>
+<wire x1="30.074" y1="18.034" x2="28.448" y2="18.034" width="0.4064" layer="1"/>
+<wire x1="28.448" y1="18.034" x2="26.67" y2="19.812" width="0.4064" layer="1"/>
+<wire x1="26.67" y1="22.86" x2="26.67" y2="25.4" width="0.8128" layer="1"/>
+</signal>
+<signal name="INT">
 <contactref element="X1" pad="2"/>
 <contactref element="X2" pad="2"/>
@@
 <wire x1="58.904" y1="64.516" x2="73.406" y2="64.516" width="0.4064" layer="1"/>
 <wire x1="73.406" y1="64.516" x2="74.92" y2="66.03" width="0.4064" layer="1"/>
-<wire x1="76.2" y1="30.48" x2="76.2" y2="61.722" width="0.4064" layer="1"/>
-<wire x1="76.2" y1="61.722" x2="73.406" y2="64.516" width="0.4064" layer="1"/>
 <wire x1="22.87" y1="11.19" x2="29.46" y2="17.78" width="0.8128" layer="16"/>
-<wire x1="29.46" y1="17.78" x2="48.51" y2="17.78" width="0.8128" layer="16"/>
-<contactref element="U$1" pad="D22"/>
-<wire x1="62.23" y1="25.4" x2="62.23" y2="28.956" width="0.6096" layer="1"/>
-<wire x1="62.23" y1="28.956" x2="62.992" y2="29.718" width="0.6096" layer="1"/>
-<wire x1="62.992" y1="29.718" x2="75.438" y2="29.718" width="0.6096" layer="1"/>
-<wire x1="75.438" y1="29.718" x2="76.2" y2="30.48" width="0.6096" layer="1"/>
-<wire x1="57.15" y1="17.78" x2="62.23" y2="25.4" width="0" layer="19" extent="16-16"/>
+<wire x1="29.46" y1="17.78" x2="36.83" y2="17.78" width="0.8128" layer="16"/>
+<wire x1="36.83" y1="17.78" x2="48.51" y2="17.78" width="0.8128" layer="16"/>
+<contactref element="U$1" pad="D3"/>
+<wire x1="36.83" y1="22.86" x2="36.83" y2="17.78" width="0.8128" layer="16"/>
+<wire x1="36.83" y1="22.86" x2="35.56" y2="24.13" width="0.4064" layer="16"/>
+<wire x1="35.56" y1="50.546" x2="30.988" y2="55.118" width="0.4064" layer="16"/>
+<wire x1="30.988" y1="55.118" x2="30.988" y2="58.928" width="0.4064" layer="16"/>
+<wire x1="34.036" y1="61.976" x2="53.086" y2="61.976" width="0.4064" layer="16"/>
+<wire x1="53.086" y1="61.976" x2="55.87" y2="64.76" width="0.4064" layer="16"/>
+<wire x1="55.87" y1="64.76" x2="55.87" y2="67.55" width="0.4064" layer="16"/>
+<wire x1="35.56" y1="24.13" x2="35.56" y2="50.546" width="0.4064" layer="16"/>
+<wire x1="30.988" y1="58.928" x2="34.036" y2="61.976" width="0.4064" layer="16"/>
+<contactref element="R2" pad="2"/>
+<wire x1="32.918" y1="18.034" x2="36.83" y2="21.946" width="0.8128" layer="1"/>
+<wire x1="36.83" y1="21.946" x2="36.83" y2="22.86" width="0.8128" layer="1"/>
 </signal>
 <signal name="N$14">
@@
 </drawing>
 <compatibility>
+<note version="6.3" minversion="6.2.2" severity="warning">
+Since Version 6.2.2 text objects can contain more than one line,
+which will not be processed correctly with this version.
+</note>
 <note version="8.2" severity="warning">
 Since Version 8.2, EAGLE supports online libraries. The ids
