File: dom-inteligentny/current-sensor/current-sensor.brd (EAGLE design)
At the start: 50.8 x 50.8 mm, 15 parts, among them K1 691218410002, Q1 16MHz, U1 ATMEGA328, U2 MAX487, U3 ACS712

Commit message: new files
Parts:
- added R2: (no value), eagle-ltspice:R1206
- added U$1: LM4040, dawidkulpa_dev:SOT23
- moved C3 3.99 mm to (14.5, 20.4)
Connections:
- net AREF: now also R2.1, U$1.1
- net GND: now also U$1.2
- net VCC: now also R2.2
Routing:
- net VCC: track 85.7 -> 95.1 mm
- net N$2: track 15.2 -> 23.6 mm
- net GND: track 138.5 -> 133.9 mm
- net AREF: track 4.34 -> 8.86 mm
Other:
- board text added: "CURR 1.1"
- board text added: "Falcon IoT"
- board text added: "weblogic.pl"
Changed lines of the file:
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@@
 <circle x="26.67" y="26.67" radius="25.4" width="0.1524" layer="20"/>
 <hole x="39.751" y="20.574" drill="3.5052"/>
-<hole x="11.049" y="17.018" drill="3.5052"/>
+<hole x="10.414" y="15.494" drill="3.5052"/>
 <hole x="25.781" y="40.767" drill="3.5052"/>
+<text x="47.117" y="23.495" size="1.778" layer="16" rot="MR0">Falcon IoT</text>
+<text x="45.974" y="12.573" size="1.778" layer="16" rot="MR0">weblogic.pl</text>
+<text x="46.482" y="16.256" size="1.778" layer="16" rot="MR0">CURR 1.1</text>
 </plain>
 <attributes>
@@
 </element>
 <element name="C2" library="adafruit" package="C1206" value="22pF" x="6.731" y="33.401" smashed="yes" rot="R270">
-<attribute name="NAME" x="7.747" y="38.227" size="1.27" layer="25" rot="R270"/>
-</element>
-<element name="C3" library="adafruit" package="C0805" value="0.1uF" x="18.415" y="21.082" smashed="yes">
-<attribute name="NAME" x="12.573" y="20.32" size="1.27" layer="25"/>
+<attribute name="NAME" x="3.81" y="32.512" size="1.27" layer="25" rot="R270"/>
+</element>
+<element name="C3" library="adafruit" package="C0805" value="0.1uF" x="14.478" y="20.447" smashed="yes">
+<attribute name="NAME" x="9.906" y="19.685" size="1.27" layer="25"/>
 </element>
 <element name="C5" library="adafruit" package="C0805" value="0.1uF" x="18.415" y="23.876" smashed="yes">
@@
 </element>
 <element name="Q1" library="crystal" package="HC49/S" value="16MHz" x="10.795" y="30.734" smashed="yes" rot="R90">
-<attribute name="NAME" x="11.43" y="22.225" size="1.27" layer="25" ratio="10" rot="R90"/>
+<attribute name="NAME" x="10.414" y="37.338" size="1.27" layer="25" ratio="10" rot="R90"/>
 </element>
 <element name="R1" library="adafruit" package="R1206" value="10K" x="29.21" y="32.258" smashed="yes">
@@
 <element name="C7" library="adafruit" package="C0805" value="0.1uF" x="22.479" y="44.45" smashed="yes" rot="R180">
 <attribute name="NAME" x="27.559" y="44.45" size="1.27" layer="25" rot="R180"/>
+</element>
+<element name="U$1" library="dawidkulpa_dev" package="SOT23" value="LM4040" x="18.669" y="20.828" smashed="yes" rot="R270">
+<attribute name="NAME" x="18.161" y="16.764" size="1.27" layer="25"/>
+</element>
+<element name="R2" library="eagle-ltspice" library_urn="urn:adsk.eagle:library:217" package="R1206" package3d_urn="urn:adsk.eagle:package:13301/1" value="" x="13.716" y="23.876" smashed="yes" rot="R180">
+<attribute name="NAME" x="10.668" y="24.003" size="1.27" layer="25" rot="R180"/>
+<attribute name="SPICEMODEL" value="NONE" x="13.716" y="23.876" size="1.778" layer="27" rot="R180" display="off"/>
+<attribute name="SPICEPREFIX" value="R" x="13.716" y="23.876" size="1.778" layer="27" rot="R180" display="off"/>
+<attribute name="VALUE" x="14.986" y="26.416" size="1.27" layer="27" rot="R180"/>
 </element>
 </elements>
@@
 <wire x1="4.953" y1="36.195" x2="9.144" y2="40.386" width="0.508" layer="1"/>
 <wire x1="9.144" y1="40.386" x2="13.716" y2="40.386" width="0.508" layer="1"/>
-<wire x1="19.265" y1="21.082" x2="19.519" y2="21.336" width="0.508" layer="1"/>
-<wire x1="19.519" y1="21.336" x2="27.94" y2="21.336" width="0.508" layer="1"/>
-<wire x1="27.94" y1="21.336" x2="28.575" y2="21.971" width="0.508" layer="1"/>
-<wire x1="28.575" y1="21.971" x2="28.575" y2="24.065" width="0.508" layer="1"/>
 <contactref element="C7" pad="2"/>
 <wire x1="21.629" y1="44.45" x2="21.629" y2="47.41" width="0.508" layer="1"/>
 <wire x1="21.629" y1="47.41" x2="21.717" y2="47.498" width="0.508" layer="1"/>
+<contactref element="U$1" pad="2"/>
+<wire x1="18.7134" y1="21.47529375" x2="18.7134" y2="21.0224" width="0.4064" layer="1"/>
+<wire x1="18.7134" y1="21.0224" x2="17.569" y2="19.878" width="0.4064" layer="1"/>
+<wire x1="19.265" y1="23.876" x2="19.265" y2="22.02689375" width="0.4064" layer="1"/>
+<wire x1="19.265" y1="22.02689375" x2="18.7134" y2="21.47529375" width="0.4064" layer="1"/>
+<wire x1="15.328" y1="20.447" x2="15.897" y2="19.878" width="0.508" layer="1"/>
+<wire x1="15.897" y1="19.878" x2="17.569" y2="19.878" width="0.508" layer="1"/>
 </signal>
 <signal name="VCC">
@@
 <wire x1="38.481" y1="35.56" x2="41.91" y2="35.56" width="0.508" layer="1"/>
 <wire x1="17.977" y1="34.792" x2="17.977" y2="36.2966" width="0.508" layer="1"/>
-<wire x1="17.177" y1="27.7114" x2="17.177" y2="26.321" width="0.508" layer="1"/>
-<wire x1="15.748" y1="24.892" x2="15.748" y2="21.463" width="0.508" layer="1"/>
-<wire x1="15.748" y1="21.463" x2="17.184" y2="21.463" width="0.508" layer="1"/>
-<wire x1="17.184" y1="21.463" x2="17.565" y2="21.082" width="0.508" layer="1"/>
-<wire x1="17.177" y1="26.321" x2="15.748" y2="24.892" width="0.508" layer="1"/>
-<wire x1="17.565" y1="21.082" x2="17.565" y2="21.756" width="0.508" layer="1"/>
-<wire x1="18.288" y1="22.479" x2="23.495" y2="22.479" width="0.508" layer="1"/>
+<wire x1="17.177" y1="27.7114" x2="17.177" y2="26.575" width="0.508" layer="1"/>
 <wire x1="23.495" y1="22.479" x2="24.765" y2="23.749" width="0.508" layer="1"/>
 <wire x1="24.765" y1="23.749" x2="24.765" y2="24.065" width="0.508" layer="1"/>
-<wire x1="17.565" y1="21.756" x2="18.288" y2="22.479" width="0.508" layer="1"/>
 <wire x1="19.577" y1="36.2966" x2="19.577" y2="37.611" width="0.508" layer="1"/>
 <wire x1="19.577" y1="37.611" x2="20.32" y2="38.354" width="0.508" layer="1"/>
@@
 <wire x1="23.329" y1="44.45" x2="23.749" y2="44.45" width="0.508" layer="1"/>
 <wire x1="23.749" y1="44.45" x2="24.257" y2="43.942" width="0.508" layer="1"/>
+<contactref element="R2" pad="2"/>
+<wire x1="17.177" y1="26.575" x2="16.256" y2="25.654" width="0.508" layer="1"/>
+<wire x1="16.256" y1="25.654" x2="13.462" y2="25.654" width="0.508" layer="1"/>
+<wire x1="13.462" y1="25.654" x2="12.294" y2="24.486" width="0.508" layer="1"/>
+<wire x1="12.294" y1="24.486" x2="12.294" y2="23.876" width="0.508" layer="1"/>
+<wire x1="12.294" y1="23.876" x2="12.294" y2="21.742" width="0.508" layer="1"/>
+<wire x1="12.294" y1="21.742" x2="13.589" y2="20.447" width="0.508" layer="1"/>
+<wire x1="13.589" y1="20.447" x2="13.628" y2="20.447" width="0.508" layer="1"/>
+<wire x1="13.628" y1="20.447" x2="13.628" y2="18.884" width="0.508" layer="1"/>
+<wire x1="13.628" y1="18.884" x2="14.097" y2="18.415" width="0.508" layer="1"/>
+<wire x1="14.097" y1="18.415" x2="19.939" y2="18.415" width="0.508" layer="1"/>
+<wire x1="19.939" y1="18.415" x2="23.495" y2="21.971" width="0.508" layer="1"/>
+<wire x1="23.495" y1="21.971" x2="23.495" y2="22.479" width="0.508" layer="1"/>
 </signal>
 <signal name="RST">
@@
 <wire x1="17.565" y1="25.185" x2="17.565" y2="23.876" width="0.508" layer="1"/>
 <wire x1="18.777" y1="26.397" x2="17.565" y2="25.185" width="0.508" layer="1"/>
+<contactref element="U$1" pad="1"/>
+<contactref element="R2" pad="1"/>
+<wire x1="17.569" y1="21.778" x2="17.569" y2="23.872" width="0.4064" layer="1"/>
+<wire x1="17.569" y1="23.872" x2="17.565" y2="23.876" width="0.4064" layer="1"/>
+<wire x1="17.565" y1="23.876" x2="15.138" y2="23.876" width="0.508" layer="1"/>
 </signal>
 <signal name="A">
@@
 <contactref element="U3" pad="2"/>
 <contactref element="K1" pad="1"/>
-<wire x1="24.765" y1="19.115" x2="22.86" y2="17.21" width="1.27" layer="1"/>
-<wire x1="22.86" y1="17.21" x2="22.86" y2="11.43" width="1.27" layer="1"/>
 <wire x1="25.4" y1="19.115" x2="26.035" y2="19.115" width="0.508" layer="1"/>
 <wire x1="24.765" y1="19.115" x2="25.211" y2="19.115" width="0.508" layer="1"/>
@@
 <wire x1="25.146" y1="18.415" x2="25.4" y2="18.669" width="0.508" layer="1"/>
 <wire x1="25.4" y1="18.669" x2="25.4" y2="19.115" width="0.508" layer="1"/>
+<wire x1="24.765" y1="19.115" x2="22.86" y2="17.21" width="2.54" layer="1"/>
+<wire x1="22.86" y1="17.21" x2="22.86" y2="11.43" width="2.54" layer="1"/>
 </signal>
 <signal name="N$2">
@@
 <wire x1="27.432" y1="18.542" x2="27.432" y2="19.812" width="0.508" layer="1"/>
 <wire x1="27.432" y1="19.812" x2="28.448" y2="19.812" width="0.508" layer="1"/>
+<wire x1="28.575" y1="19.115" x2="30.48" y2="17.21" width="2.54" layer="1"/>
+<wire x1="30.48" y1="17.21" x2="30.48" y2="11.43" width="2.54" layer="1"/>
 </signal>
 <signal name="N$3">
