File: dom-inteligentny/current-sensor/current-sensor.sch (EAGLE design)
At the start: 15 parts, among them K1 691218410002, Q1 16MHz, U1 ATMEGA328, U2 MAX487, U3 ACS712

Commit message: new files
Parts:
- added R2: (no value), eagle-ltspice:RR1206
- added U$1: LM4040, dawidkulpa_dev:LM4040
Connections:
- net AREF: now also R2.1, U$1.CATHODE
- net GND: now also U$1.ANODE
- net VCC: now also R2.2
Other:
- moved on the sheet: C5
Changed lines of the file:
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@@
 <part name="GND5" library="SparkFun" deviceset="GND" device=""/>
 <part name="P+5" library="SparkFun" deviceset="VCC" device=""/>
+<part name="U$1" library="dawidkulpa_dev" deviceset="LM4040" device=""/>
+<part name="R2" library="eagle-ltspice" library_urn="urn:adsk.eagle:library:217" deviceset="R" device="R1206" package3d_urn="urn:adsk.eagle:package:13301/1"/>
 </parts>
 <sheets>
@@
 <attribute name="VALUE" x="138.684" y="211.836" size="1.778" layer="96"/>
 </instance>
-<instance part="C5" gate="G$1" x="180.34" y="152.4" smashed="yes">
-<attribute name="NAME" x="181.356" y="153.035" size="1.778" layer="95"/>
-<attribute name="VALUE" x="181.356" y="148.209" size="1.778" layer="96"/>
-</instance>
-<instance part="GND4" gate="1" x="180.34" y="142.24" smashed="yes">
-<attribute name="VALUE" x="177.8" y="139.7" size="1.778" layer="96"/>
+<instance part="C5" gate="G$1" x="116.84" y="162.56" smashed="yes">
+<attribute name="NAME" x="117.856" y="163.195" size="1.778" layer="95"/>
+<attribute name="VALUE" x="117.856" y="158.369" size="1.778" layer="96"/>
+</instance>
+<instance part="GND4" gate="1" x="116.84" y="139.7" smashed="yes">
+<attribute name="VALUE" x="114.3" y="137.16" size="1.778" layer="96"/>
 </instance>
 <instance part="GND6" gate="1" x="101.6" y="190.5" smashed="yes">
@@
 <instance part="P+5" gate="1" x="116.84" y="210.82" smashed="yes">
 <attribute name="VALUE" x="115.824" y="214.376" size="1.778" layer="96"/>
+</instance>
+<instance part="U$1" gate="G$1" x="106.68" y="157.48" smashed="yes"/>
+<instance part="R2" gate="G$1" x="139.7" y="177.8" smashed="yes">
+<attribute name="NAME" x="135.89" y="179.2986" size="1.778" layer="95"/>
+<attribute name="VALUE" x="135.89" y="174.498" size="1.778" layer="96"/>
 </instance>
 </instances>
@@
 <segment>
 <pinref part="C5" gate="G$1" pin="2"/>
-<wire x1="180.34" y1="147.32" x2="180.34" y2="144.78" width="0.1524" layer="91"/>
+<wire x1="116.84" y1="157.48" x2="116.84" y2="144.78" width="0.1524" layer="91"/>
 <pinref part="GND4" gate="1" pin="GND"/>
+<pinref part="U$1" gate="G$1" pin="ANODE"/>
+<wire x1="116.84" y1="144.78" x2="116.84" y2="142.24" width="0.1524" layer="91"/>
+<wire x1="106.68" y1="149.86" x2="106.68" y2="144.78" width="0.1524" layer="91"/>
+<wire x1="106.68" y1="144.78" x2="116.84" y2="144.78" width="0.1524" layer="91"/>
+<junction x="116.84" y="144.78"/>
 </segment>
 <segment>
@@
 <junction x="177.8" y="182.88"/>
 <pinref part="P+1" gate="1" pin="VCC"/>
+<wire x1="177.8" y1="177.8" x2="144.78" y2="177.8" width="0.1524" layer="91"/>
+<junction x="177.8" y="177.8"/>
+<pinref part="R2" gate="G$1" pin="2"/>
 </segment>
 <segment>
@@
 <segment>
 <pinref part="U1" gate="G$1" pin="AREF"/>
-<wire x1="190.5" y1="172.72" x2="180.34" y2="172.72" width="0.1524" layer="91"/>
+<wire x1="190.5" y1="172.72" x2="116.84" y2="172.72" width="0.1524" layer="91"/>
 <pinref part="C5" gate="G$1" pin="1"/>
-<wire x1="180.34" y1="154.94" x2="180.34" y2="172.72" width="0.1524" layer="91"/>
-</segment>
-</net>
+<wire x1="116.84" y1="165.1" x2="116.84" y2="172.72" width="0.1524" layer="91"/>
+<pinref part="U$1" gate="G$1" pin="CATHODE"/>
+<wire x1="106.68" y1="165.1" x2="106.68" y2="172.72" width="0.1524" layer="91"/>
+<wire x1="106.68" y1="172.72" x2="116.84" y2="172.72" width="0.1524" layer="91"/>
+<junction x="116.84" y="172.72"/>
+<pinref part="R2" gate="G$1" pin="1"/>
+<wire x1="134.62" y1="177.8" x2="116.84" y2="177.8" width="0.1524" layer="91"/>
+<wire x1="116.84" y1="177.8" x2="116.84" y2="172.72" width="0.1524" layer="91"/>
+</segment>
+</net>
