File: dom-inteligentny/roller-shutter-bak/roller-shutter.sch (EAGLE design)
At the start: 29 parts, among them K1 RP421110, K3 691218410003, K4 RP421110, Q1 16MHz, T1 BC847, T2 BC847, U1 ATMEGA328, X1 TERMINAL-BLOCK-3.5MM-3-PIN-LO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, X2 JST-XH-05-PIN-LONG-PAD, X3 JST-XH-05-PIN-LONG-PAD

Commit message: Roller shutter
Parts:
- removed C7: (no value), eagle-ltspice:C
- removed C8, C9: (no value), eagle-ltspice:CC1812
- removed K3: 691218410003, Wurth_Elektronik_Electromechanic_Terminal_Blocks_Connectors_rev15c:691218410003
- removed R4, R5: (no value), eagle-ltspice:RR1206
- removed R6, R7: (no value), eagle-ltspice:RR2512
- removed X1: TERMINAL-BLOCK-3.5MM-3-PIN-LONG-PAD, Rembrandt Electronics - Terminal Block 3-5mm v1-0:TERMINAL-BLOCK-3.5MM-3-PIN-LONG-PAD
- removed X2, X3: JST-XH-05-PIN-LONG-PAD, Rembrandt Electronics - JST XH Connectors v1-0:JST-XH-05-PIN-LONG-PAD
- C1: value (none) -> 22pF; device rcl:CPOL-EUSANYO_SMD_C6 -> adafruit:C-USC1206
- C2: value 0.1uF -> 22pF; device adafruit:C-USC0805 -> adafruit:C-USC1206
- C3: value (none) -> 0.1uF; device eagle-ltspice:C -> adafruit:C-USC0805
- C4: value 22pF -> (none); device adafruit:C-USC1206 -> rcl:CPOL-EUSANYO_SMD_C6
- C5: value 22pF -> 0.1uF; device adafruit:C-USC1206 -> adafruit:C-USC0805
- R2, R3: device eagle-ltspice:RR1206 -> eagle-ltspice:RR1210
- renumbered K4 to K2
Connections:
- removed net N$10: C9.2, R6.1
- removed net N$4 (its old number): C8.1, C9.1, K12.P, K13.P, K22.P, K23.P, K3.3
- removed net N$7: K12.S, K13.S, K3.2, R7.2
- removed net N$8: K22.S, K23.S, K3.1, R6.2
- removed net N$9: C8.2, R7.1
- net A0: no longer R2.1
- net A1: no longer R3.1
- net A2: no longer C7.2, R5.1, X1-3.K
- net A3: no longer C3.2, R4.1, X1-2.K
- net A4: no longer X2-2.S, X3-2.S
- net A5: no longer X2-1.S, X3-1.S
- net AREF: now also C5.1; no longer C6.1
- net GND: now also C1.2, C3.2, C4.-; no longer C1.-, C3.1, C4.2, C7.1, X1-1.K, X2-4.S, X2-5.S, X3-4.S, X3-5.S
- net N$43: now also C2.1; no longer C4.1
- net N$44: now also C1.1; no longer C5.1
- net VCC: now also C3.1, C4.+, C6.1; no longer C1.+, C2.1, R4.2, R5.2, X2-3.S, X3-3.S
Other:
- moved on the sheet: C2, C3, C5, C6, D1, D2, R2, R3, T1, T2
