File: dom-inteligentny/heat-controller/controller.sch (EAGLE design)
At the start: 35 parts, among them IC1 24C64SM, IC2 DS3231/SO, K1 691218410002, K2 691218410002, K3 691218410002, T1 BC847, T10 BC847, T11 BC847, T12 BC847, T2 BC847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

Commit message: Heat controller as MCU mod
Parts:
- added C1, C2: (no value), adafruit:CPOL-US153CLV-0810
- added C3, C4: (no value), eagle-ltspice:C
- added R15: (no value), eagle-ltspice:RR1206
- added X3: TERMINAL-BLOCK-3.5MM-3-PIN-LONG-PAD, Rembrandt Electronics - Terminal Block 3-5mm v1-0:TERMINAL-BLOCK-3.5MM-3-PIN-LONG-PAD
- added X4: JST-XH-05-PIN-LONG-PAD, Rembrandt Electronics - JST XH Connectors v1-0:JST-XH-05-PIN-LONG-PAD
- added X5: GLX-S-88M, con-kycon:GLX-S-88M
- R13, R14: value 10k -> 4,7k
Connections:
- new net INT: R15.2, U$1.B0, X4-4.S, X5.2
- net 3V: now also C2.+, C4.2, R15.1
- net GND: now also C1.-, C2.-, C3.2, C4.1, X4-5.S, X5.1, X5.3
- net N$17: now also R11.1
- net SCL: now also X4-1.S, X5.4
- net SDA: now also X4-2.S, X5.6
- net VCC: now also C1.+, C3.1, X3-1.K, X3-2.K, X3-3.K, X4-3.S, X5.7, X5.8

Commit message: MLU board
Parts:
- added G1: CR2032V, battery:CR2032V
- added IC3: REG1117, burr-brown:REG1117
- added R16: R120, eagle-ltspice:RR1206
- added R17, R18: 20K, eagle-ltspice:RR1206
- IC1: value 24C64SM -> FM24CL64B
- IC2: value DS3231/SO -> DS3231
- renumbered U1 to IC4
Connections:
- removed net N$1: IC4.A, K3.1
- removed net N$2: IC4.B, K3.2
- new net A: IC4.A, K3.1, R16.1, R17.1
- new net B: IC4.B, K3.2, R16.2, R18.2
- new net N$3: G1.+, IC2.VBAT
- net 3V: now also IC3.VOUT, R17.2; no longer U$1.3.3V1
- net GND: now also G1.-, IC3.GND, R18.1
- net N$15: now also U$1.PB9; no longer U$1.PB8
- net N$16: now also U$1.PB8; no longer U$1.PB9
- net N$17: now also U$1.PA12; no longer U$1.PA11
- net N$18: now also U$1.PA11; no longer U$1.PA12
- net VCC: now also IC3.VIN
