File: e-locker/Rpi.brd (EAGLE design)
At the start: 90 x 100 mm, 6 parts

Commit message: changes
Parts:
- added E$10, E$9: (no value), adafruit:E5-8,5
- added E$11, E$12: (no value), adafruit:C0805
- added E$7, E$8: (no value), Rembrandt Electronics - JST XH Connectors v1-0:JST-XH-02-PACKAGE-LONG-PAD
Routing:
- net S$6: track 10.2 -> 85.9 mm
- net S$1: track 0.00 -> 48.0 mm
- net S$4: track 10.7 -> 40.8 mm
- net S$10: track 0.00 -> 13.6 mm
Other:
- board text added: "+"
- board text added: "24V"
