File: e-locker/simple-slave.brd (EAGLE design)
At the start: 100 x 80 mm, 38 parts, among them IC1 REG1117, Q1 16MHz, U1 ATMEGA328, U2 MAX487ESA+TCBX, X1 JST-XH-02-PIN-LONG-PAD, X10 JST-XH-04-PIN-LONG-PAD, X2 JST-XH-05-PIN-LONG-PAD, X3 JST-XH-04-PIN-LONG-PAD, X4 JST-XH-04-PIN-LONG-PAD, X5 JST-XH-04-PIN-LONG-PAD, X6 JST-XH-04-PIN-LONG-PAD, X7 JST-XH-04-PIN-LONG-PAD, X8 JST-XH-04-PIN-LONG-PAD, X9 JST-XH-04-PIN-LONG-PAD

Commit message: simple slave
Parts:
- added C7: (no value), rcl:SANYO-OSCON_SMD_C6
- added C8: 0.1uF, adafruit:C0805
- added RN1: (no value), resistor-sil:SIL9
- added U$9: (no value), zort-library:ELOCKER
- moved U$8 133.7 mm to (71.9, 65.0)
- moved X8 130.1 mm to (80.8, 32.5), turned to 90 degrees
- moved X2 129.5 mm to (50.9, 5.33)
- moved X10 127.8 mm to (80.8, 65.0), turned to 90 degrees
- moved U$7 123.1 mm to (71.9, 48.6)
- moved JP1 122.7 mm to (50.8, 64.9)
- moved U$6 114.3 mm to (71.9, 32.5)
- moved X7 113.5 mm to (80.8, 17.1), turned to 90 degrees
- moved U1 108.1 mm to (50.8, 50.8)
- moved X9 107.6 mm to (80.8, 48.6), turned to 90 degrees
- moved U$5 107.5 mm to (71.9, 17.1)
- moved R5 105.7 mm to (22.9, 20.7)
- moved C5 105.4 mm to (60.7, 50.8), turned to 90 degrees
- moved R6 104.7 mm to (65.5, 13.3), turned to 180 degrees
- moved U$1 101.9 mm to (16.5, 64.3), turned to 180 degrees
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Connections:
- removed net N$3: IC1.3
- new net N$11: U$1.P3, X3.2
- new net N$12: U$2.P3, X4.2
- new net N$13: U$3.P3, X5.2
- new net N$14: U$4.P3, X6.2
- new net N$15: U$5.P3, X7.2
- new net N$16: U$6.P3, X8.2
- new net N$18: U$7.P3, X9.2
- new net N$19: U$8.P3, X10.2
- new net V24: C4.+, C8.1, IC1.3, U$1.P2, U$2.P2, U$3.P2, U$4.P2, U$5.P2, U$6.P2, U$7.P2, U$8.P2, X1.1
- net A: now also X2.1, X2.3
- net B: now also X2.2, X2.4
- net D10: now also RN1.9, X10.4
- net D3: now also RN1.2, X3.4
- net D4: now also RN1.3, X4.4
- net D5: now also RN1.4, X5.4
- net D6: now also RN1.5, X6.4
- net D7: now also RN1.6, X7.4
- net D8: now also RN1.7, X8.4
- net D9: now also RN1.8, X9.4
- net GND: now also C7.-, C8.2, X1.2, X10.1, X10.3, X2.5, X3.1, X3.3, X4.1, X4.3, X5.1, X5.3, X6.1, X6.3, X7.1, X7.3, X8.1, X8.3, X9.1, X9.3
- net VCC: now also C7.+, RN1.1; no longer C4.+
Routing:
- net GND: track 0.00 -> 405.4 mm
- net V24: track 0.00 -> 271.4 mm, vias 0 -> 1
- net VCC: track 0.00 -> 104.0 mm, vias 0 -> 3
- net A3: track 0.00 -> 66.4 mm
- net D6: track 0.00 -> 63.7 mm
- net D10: track 0.00 -> 61.2 mm
- net D4: track 0.00 -> 60.7 mm, vias 0 -> 1
- net D3: track 0.00 -> 59.4 mm, vias 0 -> 1
- net A4: track 0.00 -> 55.8 mm, vias 0 -> 2
- net D5: track 0.00 -> 53.9 mm
- net A2: track 0.00 -> 53.0 mm
- net D7: track 0.00 -> 48.4 mm
- net D0: track 0.00 -> 45.6 mm, vias 0 -> 2
- net D1: track 0.00 -> 45.4 mm, vias 0 -> 2
- net D9: track 0.00 -> 44.5 mm
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- added copper zone on layer 1, net GND
- added copper zone on layer 16, net GND
- added copper zone on layer 1, net V24
Other:
- board size 100 x 80 mm -> 88.1 x 80 mm
- board text added: "+ -"
- board text added: "1"
- board text added: "2"
- board text added: "3"
- board text added: "4"
- board text added: "5"
- board text added: "6"
- board text added: "7"
- board text added: "8"
- board text added: "A"
- board text added: "B"
- board text added: "E-locker.pl SLAVE v1.0"
- board text added: "GND"
- board text added: "VCC"

Commit message: changes
Parts:
- removed IC1: REG1117, burr-brown:SOT223
- removed U$9: (no value), zort-library:ELOCKER
- added U$10: DC-DC-STEP-DOWN-MP1584, diy-modules:DC-DC-STEP-DOWN-MP1584
- added X11: JST-XH-02-PIN-LONG-PAD, Rembrandt Electronics - JST XH Connectors v1-0:JST-XH-02-PACKAGE-LONG-PAD
- moved C7 14.2 mm to (32.7, 36.4)
- moved C6 13.8 mm to (33.8, 42.4)
- moved X1 7.32 mm to (23.2, 5.33)
- moved C8 6.86 mm to (23.1, 11.5)
- moved R5 5.36 mm to (22.4, 26.0)
- moved C4 5.03 mm to (24.7, 17.9)
Connections:
- net GND: now also U$10.IN-.1, U$10.OUT-.1, X11.2; no longer IC1.1
- net V24: now also U$10.IN+.2; no longer IC1.3
- net VCC: now also U$10.OUT+.2, X11.1; no longer IC1.2
Routing:
- net V24: track 271.4 -> 318.4 mm, vias 1 -> 0
- net VCC: track 104.0 -> 139.0 mm
- net GND: track 405.4 -> 426.9 mm
- net A3: track 66.4 -> 62.7 mm
- net N$5: track 2.88 -> 5.65 mm
- net D6: track 63.7 -> 65.4 mm
Other:
- board text added: "24V"
- board text added: "5V + -"

Commit message: Rpi master board
Parts:
- added U$9: (no value), zort-library:ELOCKER
Changed lines of the file:
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@@
 <?xml version="1.0" encoding="utf-8"?>
 <!DOCTYPE eagle SYSTEM "eagle.dtd">
-<eagle version="9.2.2">
+<eagle version="9.6.2">
 <drawing>
 <settings>
@@
 <attribute name="NAME" x="31.051" y="3.294" size="1.016" layer="25" ratio="10" rot="R90"/>
 </element>
+<element name="U$9" library="zort-library" package="ELOCKER" value="" x="60.6044" y="2.1844" smashed="yes"/>
 </elements>
 <signals>
