File: e-locker/simple-slave.sch (EAGLE design)
At the start: 38 parts, among them IC1 REG1117, Q1 16MHz, U1 ATMEGA328, U2 MAX487ESA+TCBX, X1 JST-XH-02-PIN-LONG-PAD, X10 JST-XH-04-PIN-LONG-PAD, X2 JST-XH-05-PIN-LONG-PAD, X3 JST-XH-04-PIN-LONG-PAD, X4 JST-XH-04-PIN-LONG-PAD, X5 JST-XH-04-PIN-LONG-PAD, X6 JST-XH-04-PIN-LONG-PAD, X7 JST-XH-04-PIN-LONG-PAD, X8 JST-XH-04-PIN-LONG-PAD, X9 JST-XH-04-PIN-LONG-PAD

Commit message: simple slave
Parts:
- added C7: (no value), rcl:CPOL-EUSANYO_SMD_C6
- added C8: 0.1uF, adafruit:C-USC0805
- added RN1: (no value), resistor-sil:G08R
Connections:
- removed net N$3: IC1.VIN
- new net N$11: U$1.S, X3-2.S
- new net N$12: U$2.S, X4-2.S
- new net N$13: U$3.S, X5-2.S
- new net N$14: U$4.S, X6-2.S
- new net N$15: U$5.S, X7-2.S
- new net N$16: U$6.S, X8-2.S
- new net N$18: U$7.S, X9-2.S
- new net N$19: U$8.S, X10-2.S
- new net V24: C4.+, C8.1, IC1.VIN, U$1.D, U$2.D, U$3.D, U$4.D, U$5.D, U$6.D, U$7.D, U$8.D, X1-1.S
- net A: now also X2-1.S, X2-3.S
- net B: now also X2-2.S, X2-4.S
- net D10: now also RN1.9, X10-4.S
- net D3: now also RN1.2, X3-4.S
- net D4: now also RN1.3, X4-4.S
- net D5: now also RN1.4, X5-4.S
- net D6: now also RN1.5, X6-4.S
- net D7: now also RN1.6, X7-4.S
- net D8: now also RN1.7, X8-4.S
- net D9: now also RN1.8, X9-4.S
- net GND: now also C7.-, C8.2, X1-2.S, X10-1.S, X10-3.S, X2-5.S, X3-1.S, X3-3.S, X4-1.S, X4-3.S, X5-1.S, X5-3.S, X6-1.S, X6-3.S, X7-1.S, X7-3.S, X8-1.S, X8-3.S, X9-1.S, X9-3.S
- net VCC: now also C7.+, RN1.1; no longer C4.+
Other:
- moved on the sheet: C4, X1-1, X2-1, X2-2, X2-3, X2-4, X2-5

Commit message: changes
Parts:
- removed IC1: REG1117, burr-brown:REG1117
- added U$10: DC-DC-STEP-DOWN-MP1584, diy-modules:DC-DC-STEP-DOWN-MP1584
- added X11: JST-XH-02-PIN-LONG-PAD, Rembrandt Electronics - JST XH Connectors v1-0:JST-XH-02-PIN-LONG-PAD
Connections:
- net GND: now also U$10.IN-.1, U$10.OUT-.1, X11-2.S; no longer IC1.GND
- net V24: now also U$10.IN+.2; no longer IC1.VIN
- net VCC: now also U$10.OUT+.2, X11-1.S; no longer IC1.VOUT
Changed lines of the file:
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@@
 <?xml version="1.0" encoding="utf-8"?>
 <!DOCTYPE eagle SYSTEM "eagle.dtd">
-<eagle version="9.6.2">
+<eagle version="9.2.2">
 <drawing>
 <settings>
@@
 <part name="GND5" library="SparkFun" deviceset="GND" device=""/>
 <part name="P+7" library="SparkFun" deviceset="VCC" device=""/>
-<part name="IC1" library="burr-brown" library_urn="urn:adsk.eagle:library:111" deviceset="REG1117" device="" package3d_urn="urn:adsk.eagle:package:4940/1"/>
 <part name="U$1" library="dawidkulpa_dev" deviceset="MOSFET-N" device="TO252"/>
 <part name="U$2" library="dawidkulpa_dev" deviceset="MOSFET-N" device="TO252"/>
@@
 <part name="C7" library="rcl" library_urn="urn:adsk.eagle:library:334" deviceset="CPOL-EU" device="SANYO_SMD_C6" package3d_urn="urn:adsk.eagle:package:23465/1"/>
 <part name="C8" library="adafruit" deviceset="C-US" device="C0805" value="0.1uF"/>
+<part name="U$10" library="diy-modules" deviceset="DC-DC-STEP-DOWN-MP1584" device=""/>
+<part name="X11" library="Rembrandt Electronics - JST XH Connectors v1-0" deviceset="JST-XH-02-PIN" device="-LONG-PAD"/>
 </parts>
 <sheets>
@@
 <instance part="P+7" gate="1" x="114.3" y="210.82" smashed="yes">
 <attribute name="VALUE" x="113.284" y="214.376" size="1.778" layer="96"/>
-</instance>
-<instance part="IC1" gate="G$1" x="96.52" y="157.48" smashed="yes">
-<attribute name="NAME" x="88.9" y="163.195" size="1.778" layer="95" ratio="10"/>
-<attribute name="VALUE" x="91.44" y="160.02" size="1.778" layer="96" ratio="10"/>
 </instance>
 <instance part="U$1" gate="G$1" x="350.52" y="203.2" smashed="yes" rot="R90"/>
@@
 <attribute name="VALUE" x="287.02" y="106.045" size="1.778" layer="96"/>
 </instance>
-<instance part="GND9" gate="1" x="78.74" y="142.24" smashed="yes">
-<attribute name="VALUE" x="76.2" y="139.7" size="1.778" layer="96"/>
+<instance part="GND9" gate="1" x="71.12" y="144.78" smashed="yes">
+<attribute name="VALUE" x="68.58" y="142.24" size="1.778" layer="96"/>
 </instance>
 <instance part="GND10" gate="1" x="66.04" y="91.44" smashed="yes">
@@
 <attribute name="NAME" x="69.596" y="203.835" size="1.778" layer="95"/>
 <attribute name="VALUE" x="69.596" y="199.009" size="1.778" layer="96"/>
+</instance>
+<instance part="U$10" gate="G$1" x="93.98" y="152.4" smashed="yes" rot="MR180">
+<attribute name="NAME" x="81.28" y="137.16" size="1.778" layer="95" rot="MR180"/>
+<attribute name="VALUE" x="81.28" y="139.7" size="1.778" layer="96" rot="MR180"/>
+</instance>
+<instance part="X11" gate="-2" x="58.42" y="175.26" smashed="yes" rot="R180">
+<attribute name="NAME" x="55.88" y="176.022" size="1.524" layer="95" rot="R180"/>
+</instance>
+<instance part="X11" gate="-1" x="58.42" y="177.8" smashed="yes" rot="R180">
+<attribute name="NAME" x="55.88" y="178.562" size="1.524" layer="95" rot="R180"/>
 </instance>
 </instances>
@@
 <wire x1="132.08" y1="165.1" x2="132.08" y2="154.94" width="0.1524" layer="91"/>
 <pinref part="C1" gate="G$1" pin="2"/>
-<wire x1="132.08" y1="154.94" x2="132.08" y2="142.24" width="0.1524" layer="91"/>
+<wire x1="132.08" y1="154.94" x2="132.08" y2="147.32" width="0.1524" layer="91"/>
+<wire x1="132.08" y1="147.32" x2="132.08" y2="142.24" width="0.1524" layer="91"/>
 <wire x1="137.16" y1="154.94" x2="132.08" y2="154.94" width="0.1524" layer="91"/>
 <junction x="132.08" y="154.94"/>
 <pinref part="GND1" gate="1" pin="GND"/>
+<pinref part="U$10" gate="G$1" pin="OUT-.1"/>
+<wire x1="111.76" y1="147.32" x2="114.3" y2="147.32" width="0.1524" layer="91"/>
+<junction x="132.08" y="147.32"/>
+<pinref part="X11" gate="-2" pin="S"/>
+<wire x1="114.3" y1="147.32" x2="132.08" y2="147.32" width="0.1524" layer="91"/>
+<wire x1="60.96" y1="175.26" x2="114.3" y2="175.26" width="0.1524" layer="91"/>
+<wire x1="114.3" y1="175.26" x2="114.3" y2="147.32" width="0.1524" layer="91"/>
+<junction x="114.3" y="147.32"/>
 </segment>
 <segment>
@@
 </segment>
 <segment>
-<pinref part="IC1" gate="G$1" pin="GND"/>
-<wire x1="96.52" y1="144.78" x2="78.74" y2="144.78" width="0.1524" layer="91"/>
 <pinref part="X1" gate="-2" pin="S"/>
-<wire x1="78.74" y1="144.78" x2="60.96" y2="144.78" width="0.1524" layer="91"/>
-<wire x1="60.96" y1="152.4" x2="60.96" y2="144.78" width="0.1524" layer="91"/>
+<wire x1="71.12" y1="147.32" x2="60.96" y2="147.32" width="0.1524" layer="91"/>
+<wire x1="60.96" y1="152.4" x2="60.96" y2="147.32" width="0.1524" layer="91"/>
 <pinref part="GND9" gate="1" pin="GND"/>
-<junction x="78.74" y="144.78"/>
+<pinref part="U$10" gate="G$1" pin="IN-.1"/>
+<wire x1="71.12" y1="147.32" x2="76.2" y2="147.32" width="0.1524" layer="91"/>
+<junction x="71.12" y="147.32"/>
 </segment>
 <segment>
@@
 </segment>
 <segment>
-<pinref part="IC1" gate="G$1" pin="VOUT"/>
-<wire x1="109.22" y1="157.48" x2="114.3" y2="157.48" width="0.1524" layer="91"/>
-<label x="114.3" y="157.48" size="1.778" layer="95" xref="yes"/>
+<pinref part="U$10" gate="G$1" pin="OUT+.2"/>
+<wire x1="111.76" y1="157.48" x2="116.84" y2="157.48" width="0.1524" layer="91"/>
+<label x="119.38" y="157.48" size="1.778" layer="95" xref="yes"/>
+<pinref part="X11" gate="-1" pin="S"/>
+<wire x1="116.84" y1="157.48" x2="119.38" y2="157.48" width="0.1524" layer="91"/>
+<wire x1="60.96" y1="177.8" x2="116.84" y2="177.8" width="0.1524" layer="91"/>
+<wire x1="116.84" y1="177.8" x2="116.84" y2="157.48" width="0.1524" layer="91"/>
+<junction x="116.84" y="157.48"/>
 </segment>
 </net>
@@
 <net name="V24" class="0">
 <segment>
-<pinref part="IC1" gate="G$1" pin="VIN"/>
-<wire x1="83.82" y1="157.48" x2="60.96" y2="157.48" width="0.1524" layer="91"/>
 <pinref part="X1" gate="-1" pin="S"/>
 <wire x1="60.96" y1="154.94" x2="60.96" y2="157.48" width="0.1524" layer="91"/>
 <label x="68.58" y="157.48" size="1.778" layer="95" rot="R90" xref="yes"/>
-</segment>
-<segment>
+<pinref part="U$10" gate="G$1" pin="IN+.2"/>
+<wire x1="60.96" y1="157.48" x2="76.2" y2="157.48" width="0.1524" layer="91"/>
+</segment>
+<segment>

Commit message: incorrect mosfets - WIP
Parts:
- removed U$1: (no value), dawidkulpa_dev:MOSFET-NTO252
- added Q2: SPD30P06PTO252, transistor-fet:SPD30P06PTO252
Connections:
- net N$1: now also Q2.G; no longer U$1.G
- net N$11: now also Q2.D; no longer U$1.S
- net V24: now also Q2.S; no longer U$1.D
Changed lines of the file:
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@@
 <?xml version="1.0" encoding="utf-8"?>
 <!DOCTYPE eagle SYSTEM "eagle.dtd">
-<eagle version="9.2.2">
+<eagle version="9.6.2">
 <drawing>
 <settings>
@@
 <part name="GND5" library="SparkFun" deviceset="GND" device=""/>
 <part name="P+7" library="SparkFun" deviceset="VCC" device=""/>
-<part name="U$1" library="dawidkulpa_dev" deviceset="MOSFET-N" device="TO252"/>
 <part name="U$2" library="dawidkulpa_dev" deviceset="MOSFET-N" device="TO252"/>
 <part name="U$3" library="dawidkulpa_dev" deviceset="MOSFET-N" device="TO252"/>
@@
 <part name="U$10" library="diy-modules" deviceset="DC-DC-STEP-DOWN-MP1584" device=""/>
 <part name="X11" library="Rembrandt Electronics - JST XH Connectors v1-0" deviceset="JST-XH-02-PIN" device="-LONG-PAD"/>
+<part name="Q2" library="transistor-fet" library_urn="urn:adsk.eagle:library:396" deviceset="SPD30P06P" device="TO252" package3d_urn="urn:adsk.eagle:package:28537/2"/>
 </parts>
 <sheets>
@@
 <attribute name="VALUE" x="113.284" y="214.376" size="1.778" layer="96"/>
 </instance>
-<instance part="U$1" gate="G$1" x="350.52" y="203.2" smashed="yes" rot="R90"/>
 <instance part="U$2" gate="G$1" x="350.52" y="185.42" smashed="yes" rot="R90"/>
 <instance part="U$3" gate="G$1" x="350.52" y="167.64" smashed="yes" rot="R90"/>
@@
 <instance part="X11" gate="-1" x="58.42" y="177.8" smashed="yes" rot="R180">
 <attribute name="NAME" x="55.88" y="178.562" size="1.524" layer="95" rot="R180"/>
+</instance>
+<instance part="Q2" gate="G$1" x="350.52" y="203.2" smashed="yes">
+<attribute name="NAME" x="339.09" y="201.93" size="1.778" layer="95"/>
 </instance>
 </instances>
@@
 </segment>
 <segment>
-<pinref part="U$1" gate="G$1" pin="D"/>
 <wire x1="353.06" y1="208.28" x2="353.06" y2="210.82" width="0.1524" layer="91"/>
 <wire x1="353.06" y1="210.82" x2="330.2" y2="210.82" width="0.1524" layer="91"/>
 <label x="330.2" y="210.82" size="1.778" layer="95" rot="R180" xref="yes"/>
+<pinref part="Q2" gate="G$1" pin="S"/>
 </segment>
 <segment>
@@
 </segment>
 </net>
-<net name="N$1" class="0">
-<segment>
-<pinref part="U$1" gate="G$1" pin="G"/>
-<pinref part="R2" gate="G$1" pin="1"/>
-</segment>
-</net>
 <net name="N$2" class="0">
 <segment>
@@
 <wire x1="391.16" y1="205.74" x2="358.14" y2="205.74" width="0.1524" layer="91"/>
 <wire x1="358.14" y1="205.74" x2="358.14" y2="198.12" width="0.1524" layer="91"/>
-<pinref part="U$1" gate="G$1" pin="S"/>
 <wire x1="358.14" y1="198.12" x2="353.06" y2="198.12" width="0.1524" layer="91"/>
+<pinref part="Q2" gate="G$1" pin="D"/>
 </segment>
 </net>
@@
 </segment>
 </net>
+<net name="N$1" class="0">
+<segment>
+<pinref part="R2" gate="G$1" pin="1"/>
+<pinref part="Q2" gate="G$1" pin="G"/>
+<wire x1="347.98" y1="203.2" x2="347.98" y2="205.74" width="0.1524" layer="91"/>
+</segment>
+</net>
