File: e-locker/slave-16.brd (EAGLE design)
At the start: 93.3 x 100 mm, 118 parts, among them IC1 PCF8574P, IC2 PCF8574P, IC3 PCF8574P, IC4 PCF8574P, Q1 BC547B, Q2 BC547B, Q3 BC547B, Q4 BC547B, Q5 BC547B, Q6 BC547B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

Commit message: slave 16
Parts:
- R1, R35, R36: value (none) -> 1k
Other:
- board text added: "VCC"
