File: e-locker/slave-16.sch (EAGLE design)
At the start: 117 parts, among them IC1 PCF8574P, IC2 PCF8574P, IC3 PCF8574P, IC4 PCF8574P, Q1 BC547B, Q2 BC547B, Q3 BC547B, Q4 BC547B, Q5 BC547B, Q6 BC547B, Q7 BC547B, Q8 BC547B, T1 BC547, T2 BC547, T3 BC547, T4 BC547, T5 BC547, T6 BC547, T7 BC547, T8 BC547, X1 JST-XH-02-PIN-LONG-PAD, X10 JST-XH-04-PIN-LONG-PAD, X11 JST-XH-02-PIN-LONG-PAD, X12 JST-XH-04-PIN-LONG-PAD, X13 JST-XH-04-PIN-LONG-PAD, X14 JST-XH-04-PIN-LONG-PAD, X15 JST-XH-04-PIN-LONG-PAD, X16 JST-XH-04-PIN-LONG-PAD, X17 JST-XH-04-PIN-LONG-PAD, X18 JST-XH-04-PIN-LONG-PAD, X19 JST-XH-04-PIN-LONG-PAD, X2 JST-XH-05-PIN-LONG-PAD, X20 JST-XH-05-PIN-LONG-PAD, X21 JST-XH-02-PIN-LONG-PAD, X22 JST-XH-02-PIN-LONG-PAD, X3 JST-XH-04-PIN-LONG-PAD, X4 JST-XH-04-PIN-LONG-PAD, X5 JST-XH-04-PIN-LONG-PAD, X6 JST-XH-04-PIN-LONG-PAD, X7 JST-XH-04-PIN-LONG-PAD, X8 JST-XH-04-PIN-LONG-PAD, X9 JST-XH-04-PIN-LONG-PAD

Commit message: slave 16
Parts:
- R1, R35, R36: value (none) -> 1k
Changed lines of the file:
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@@
 <part name="U$18" library="mosfet" deviceset="IRLML6402" device=""/>
 <part name="U$19" library="mosfet" deviceset="IRLML6402" device=""/>
-<part name="R1" library="eagle-ltspice" library_urn="urn:adsk.eagle:library:217" deviceset="R" device="R1206" package3d_urn="urn:adsk.eagle:package:13301/1"/>
+<part name="R1" library="eagle-ltspice" library_urn="urn:adsk.eagle:library:217" deviceset="R" device="R1206" package3d_urn="urn:adsk.eagle:package:13301/1" value="1k"/>
 <part name="R10" library="eagle-ltspice" library_urn="urn:adsk.eagle:library:217" deviceset="R" device="R1206" package3d_urn="urn:adsk.eagle:package:13301/1"/>
 <part name="R11" library="eagle-ltspice" library_urn="urn:adsk.eagle:library:217" deviceset="R" device="R1206" package3d_urn="urn:adsk.eagle:package:13301/1"/>
@@
 <part name="GND30" library="supply1" library_urn="urn:adsk.eagle:library:371" deviceset="GND" device=""/>
 <part name="GND31" library="supply1" library_urn="urn:adsk.eagle:library:371" deviceset="GND" device=""/>
-<part name="R35" library="eagle-ltspice" library_urn="urn:adsk.eagle:library:217" deviceset="R" device="R1206" package3d_urn="urn:adsk.eagle:package:13301/1"/>
-<part name="R36" library="eagle-ltspice" library_urn="urn:adsk.eagle:library:217" deviceset="R" device="R1206" package3d_urn="urn:adsk.eagle:package:13301/1"/>
+<part name="R35" library="eagle-ltspice" library_urn="urn:adsk.eagle:library:217" deviceset="R" device="R1206" package3d_urn="urn:adsk.eagle:package:13301/1" value="1k"/>
+<part name="R36" library="eagle-ltspice" library_urn="urn:adsk.eagle:library:217" deviceset="R" device="R1206" package3d_urn="urn:adsk.eagle:package:13301/1" value="1k"/>
 <part name="R37" library="eagle-ltspice" library_urn="urn:adsk.eagle:library:217" deviceset="R" device="R1206" package3d_urn="urn:adsk.eagle:package:13301/1"/>
 <part name="R38" library="eagle-ltspice" library_urn="urn:adsk.eagle:library:217" deviceset="R" device="R1206" package3d_urn="urn:adsk.eagle:package:13301/1"/>
