File: e-locker/master-sim800.brd (EAGLE design)
At the start: 100 x 100 mm, 48 parts, among them T1 BC847, T2 BC847, T3 BC847, U1 AT24C128C-SSHM-T, X1 JST-XH-02-PIN-LONG-PAD, X10 JST-XH-05-PIN-LONG-PAD, X11 JST-XH-02-PIN-LONG-PAD, X12 JST-XH-02-PIN-LONG-PAD, X13 JST-XH-02-PIN-LONG-PAD, X2 JST-XH-02-PIN-LONG-PAD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

Commit message: master new revision
Parts:
- added C12, C13: (no value), adafruit:E5-8,5
- added R12: (no value), eagle-ltspice:R1206
- added R13, R14: 1k, eagle-ltspice:R1206
- added R15, R16: 5.6k, eagle-ltspice:R1206
- added T4: BC847, transistor:SOT23
- added U$7: SIM800L-V1, SIM800L:SIM800L
- added U$8: DC-DC-STEP-DOWN-MP2307, diy-modules:DC-DC-STEP-DOWN-MP2307
Connections:
- new net N$18: T4.3, U$2.7, U$7.RESET
- new net N$24: R12.1, U$1.GPIO5
- new net N$25: R12.2, T4.1
- new net N$26: R13.2, U$7.RXD
- new net N$27: R14.2, U$7.TXD
- new net N$28: C12.+, C13.+, U$7.4V, U$8.OUT+
- net GND: now also C12.-, C13.-, R15.2, R16.2, T4.2, U$7.GND, U$8.IN-, U$8.OUT-
- net N$23: now also U$8.IN+
- net N$3: now also R14.1, R15.1
- net N$4: now also R13.1, R16.1
Routing:
- net GND: track 524.0 -> 625.7 mm
- net N$28: track 0.00 -> 71.3 mm
- net N$23: track 72.6 -> 139.0 mm
- net N$18: track 0.00 -> 53.1 mm
- net N$3: track 50.0 -> 101.5 mm, vias 0 -> 1
- net N$4: track 43.4 -> 84.2 mm, vias 0 -> 1
- net N$27: track 0.00 -> 21.3 mm
- net N$24: track 0.00 -> 17.4 mm
- net N$25: track 0.00 -> 13.7 mm
- net N$26: track 0.00 -> 4.34 mm
- net VCC: track 261.0 -> 262.6 mm
Other:
- board text added: "E-LOCKER.pl MASTER 3G rev. 1.2"
- board text removed: "E-LOCKER.pl MASTER 3G rev. 1.1"
