File: e-locker/master-sim800.brd (EAGLE design)
At the start: 100 x 100 mm, 58 parts, among them T1 BC847, T2 BC847, T3 BC847, T4 BC847, U1 AT24C128C-SSHM-T, X1 JST-XH-02-PIN-LONG-PAD, X10 JST-XH-05-PIN-LONG-PAD, X11 JST-XH-02-PIN-LONG-PAD, X12 JST-XH-02-PIN-LONG-PAD, X13 JST-XH-02-PIN-LONG-PAD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

Commit message: changes
Routing:
- net GND: track 625.7 -> 641.2 mm
Changed lines of the file:
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@@
 <wire x1="75.921" y1="89.662" x2="75.921" y2="88.115" width="0.8128" layer="1"/>
 <wire x1="75.921" y1="88.115" x2="77.041" y2="86.995" width="0.8128" layer="1"/>
+<wire x1="73.406" y1="83.693" x2="73.406" y2="68.199" width="2.54" layer="16"/>
 </signal>
 <signal name="N$2">
