File: e-locker/slave-16-mosfet.brd (EAGLE design)
At the start: 93.3 x 100 mm, 134 parts, among them IC1 PCF8574P, IC2 PCF8574P, IC3 PCF8574P, IC4 PCF8574P, Q1 BC547B, Q2 BC547B, Q3 BC547B, Q4 BC547B, Q5 BC547B, Q6 BC547B, Q7 BC547B, Q8 BC547B, T1 BC547, T2 BC547, T3 BC547, T4 BC547, T5 BC547, T6 BC547, T7 BC547, T8 BC547, X1 JST-XH-02-PIN-LONG-PAD, X10 JST-XH-04-PIN-LONG-PAD, X11 JST-XH-02-PIN-LONG-PAD, X12 JST-XH-04-PIN-LONG-PAD, X13 JST-XH-04-PIN-LONG-PAD, X14 JST-XH-04-PIN-LONG-PAD, X15 JST-XH-04-PIN-LONG-PAD, X16 JST-XH-04-PIN-LONG-PAD, X17 JST-XH-04-PIN-LONG-PAD, X18 JST-XH-04-PIN-LONG-PAD, X19 JST-XH-04-PIN-LONG-PAD, X2 JST-XH-05-PIN-LONG-PAD, X20 JST-XH-05-PIN-LONG-PAD, X21 JST-XH-02-PIN-LONG-PAD, X22 JST-XH-02-PIN-LONG-PAD, X3 JST-XH-04-PIN-LONG-PAD, X4 JST-XH-04-PIN-LONG-PAD, X5 JST-XH-04-PIN-LONG-PAD, X6 JST-XH-04-PIN-LONG-PAD, X7 JST-XH-04-PIN-LONG-PAD, X8 JST-XH-04-PIN-LONG-PAD, X9 JST-XH-04-PIN-LONG-PAD

Commit message: WIP
Parts:
- moved U$1 433.8 mm to (9.40, 84.8), turned to 90 degrees
- moved U$2 404.4 mm to (9.40, 73.2), turned to 90 degrees
- moved U$3 373.8 mm to (9.27, 60.3), turned to 90 degrees
- moved U$4 343.0 mm to (9.27, 47.4), turned to 90 degrees
- moved U$7 332.7 mm to (19.6, 90.3)
- moved U$8 315.4 mm to (32.1, 90.3)
- moved U$5 312.9 mm to (9.27, 35.1), turned to 90 degrees
- moved U$6 282.9 mm to (9.27, 22.7), turned to 90 degrees
- moved U$17 245.1 mm to (94.9, 59.8), turned to 90 degrees
- moved R59 120.1 mm to (16.8, 82.2), turned to 180 degrees
- moved R56 115.9 mm to (97.2, 51.6)
- moved R51 111.2 mm to (42.2, 102.4)
- moved R60 106.6 mm to (16.5, 64.5), turned to 180 degrees
- moved R61 104.5 mm to (15.6, 58.3), turned to 90 degrees
- moved R62 94.9 mm to (16.5, 44.5), turned to 180 degrees
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Connections:
- removed net N$11: R43.1, U$1.G
- new net N$81: R43.1, R59.2, U$1.G
- net N$12: now also R60.2
- net N$13: now also R61.2
- net N$14: now also R62.2
- net N$56: now also R66.2
- net N$59: now also R65.2
- net N$63: now also R64.2
- net N$64: now also R63.2
- net V24: no longer R59.2, R60.2, R61.2, R62.2, R63.2, R64.2, R65.2, R66.2
Routing:
- net GND: track 922.0 -> 806.2 mm
- net VCC: track 326.7 -> 226.2 mm
- net A5: track 168.1 -> 88.9 mm, vias 3 -> 1
- net A4: track 161.9 -> 101.3 mm, vias 2 -> 3
- net P7: track 69.6 -> 11.1 mm
- net N$75: track 0.00 -> 34.1 mm
- net V24: track 228.1 -> 254.8 mm
- net N$63: track 35.9 -> 11.4 mm
- net N$37: track 23.9 -> 0.00 mm
- net N$76: track 0.00 -> 21.3 mm
- net N$36: track 20.3 -> 0.00 mm
- net N$64: track 24.2 -> 8.10 mm
- net P6: track 74.5 -> 90.6 mm, vias 0 -> 1
- net P2: track 41.9 -> 56.4 mm, vias 0 -> 1
- net N$12: track 1.08 -> 12.2 mm
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
Commit message: new master and slave16 changes
Parts:
- removed JP2: (no value), pinhead-zmiany-JP:2X08
- added JP3: (no value), adafruit:2X04
- added U$11: (no value), logo:CE_7.3MM
- moved U$19 250.8 mm to (84.3, 33.7), turned to 270 degrees
- moved U$18 246.4 mm to (84.3, 46.9), turned to 270 degrees
- moved U$16 236.7 mm to (84.2, 72.3), turned to 270 degrees
- moved U$15 231.7 mm to (84.2, 84.8), turned to 270 degrees
- moved U$14 215.9 mm to (70.7, 90.2)
- moved U$13 195.5 mm to (57.9, 90.2)
- moved U$12 175.4 mm to (45.1, 90.2)
- moved R66 150.0 mm to (34.0, 81.0), turned to 90 degrees
- moved R65 147.2 mm to (22.1, 83.8), turned to 180 degrees
- moved R54 122.6 mm to (77.3, 85.9), turned to 270 degrees
- moved R55 116.2 mm to (76.5, 74.5), turned to 90 degrees
- moved R57 108.8 mm to (72.3, 60.1), turned to 90 degrees
- moved R53 108.8 mm to (64.6, 81.7), turned to 180 degrees
- moved R58 108.5 mm to (72.9, 55.1), turned to 180 degrees
- moved R52 101.4 mm to (54.1, 83.1), turned to 270 degrees
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Connections:
- net GND: now also JP3.2, JP3.4, JP3.6, JP3.8; no longer JP2.10, JP2.12, JP2.14, JP2.16, JP2.2, JP2.4, JP2.6, JP2.8
- net N$10: no longer JP2.15
- net N$17: no longer JP2.13
- net N$20: no longer JP2.11
- net N$21: no longer JP2.9
- net N$22: now also JP3.7; no longer JP2.7
- net N$23: now also JP3.5; no longer JP2.5
- net N$24: now also JP3.3; no longer JP2.3
- net N$25: now also JP3.1; no longer JP2.1
Routing:
- net V24: track 254.8 -> 361.7 mm
- net P7: track 11.1 -> 82.1 mm, vias 0 -> 1
- net VCC: track 226.2 -> 276.2 mm, vias 2 -> 5
- net GND: track 806.2 -> 850.2 mm, vias 0 -> 2
- net S15: track 53.4 -> 20.2 mm
- net S14: track 39.9 -> 12.1 mm
- net A5: track 88.9 -> 111.6 mm
- net N$2: track 0.00 -> 22.3 mm
- net P8: track 90.3 -> 74.7 mm
- net P15: track 21.1 -> 36.5 mm, vias 0 -> 2
- net N$61: track 2.75 -> 16.9 mm
- net P4: track 35.2 -> 47.8 mm
- net P10: track 61.6 -> 73.7 mm, vias 1 -> 2
- net N$3: track 15.8 -> 3.92 mm
- net N$56: track 0.00 -> 11.9 mm
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Other:
- board text added: "2022"
- board text added: "E-locker.pl SLAVE rev 2.1"
- board text added: "JLCJLCJLCJLC"
- board text removed: "E-locker.pl SLAVE rev 2.0"

Commit message: mosfet slave fix
Parts:
- R51, R64: value (none) -> 2,2k
Routing:
- net D0: track 29.4 -> 30.5 mm
Other:
- board text added: "E-locker.pl SLAVE rev 2.2"
- board text removed: "E-locker.pl SLAVE rev 2.1"
Changed lines of the file:
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@@
 <text x="9.0424" y="9.4742" size="1.27" layer="25">E-locker.pl
 SLAVE
-rev 2.1</text>
+rev 2.2</text>
 <text x="9.144" y="0.508" size="2.54" layer="21" font="vector">+    -</text>
 <text x="52.832" y="0.889" size="1.27" layer="21" font="vector">A</text>
@@
 <attribute name="POPULARITY" value="47" x="36.703" y="73.279" size="1.778" layer="27" display="off"/>
 </element>
-<element name="R51" library="eagle-ltspice" library_urn="urn:adsk.eagle:library:217" package="R1206" package3d_urn="urn:adsk.eagle:package:13301/1" value="" x="42.164" y="83.058" smashed="yes" rot="R270">
+<element name="R51" library="eagle-ltspice" library_urn="urn:adsk.eagle:library:217" package="R1206" package3d_urn="urn:adsk.eagle:package:13301/1" value="2,2k" x="42.164" y="83.058" smashed="yes" rot="R270">
 <attribute name="NAME" x="43.434" y="85.09" size="1.27" layer="25" rot="R270"/>
 <attribute name="SPICEMODEL" value="NONE" x="42.164" y="83.058" size="1.778" layer="27" rot="R270" display="off"/>
@@
 <attribute name="VALUE" x="13.716" y="35.306" size="1.27" layer="27" rot="R270"/>
 </element>
-<element name="R64" library="eagle-ltspice" library_urn="urn:adsk.eagle:library:217" package="R1206" package3d_urn="urn:adsk.eagle:package:13301/1" value="" x="18.796" y="21.717" smashed="yes" rot="R270">
+<element name="R64" library="eagle-ltspice" library_urn="urn:adsk.eagle:library:217" package="R1206" package3d_urn="urn:adsk.eagle:package:13301/1" value="2,2k" x="18.796" y="21.717" smashed="yes" rot="R270">
 <attribute name="NAME" x="16.256" y="22.86" size="1.27" layer="25" rot="R270"/>
 <attribute name="SPICEMODEL" value="NONE" x="18.796" y="21.717" size="1.778" layer="27" rot="R270" display="off"/>
@@
 <signal name="D0">
 <contactref element="U$10" pad="RX"/>
-<wire x1="43.3106" y1="16.1026" x2="57.912" y2="30.704" width="0.508" layer="1"/>
-<wire x1="57.912" y1="30.704" x2="57.912" y2="36.957" width="0.508" layer="1"/>
+<wire x1="57.912" y1="28.799" x2="45.2156" y2="16.1026" width="0.508" layer="1"/>
+<wire x1="43.3106" y1="16.1026" x2="45.2156" y2="16.1026" width="0.508" layer="1"/>
+<wire x1="57.912" y1="28.799" x2="57.912" y2="36.957" width="0.508" layer="1"/>
 <wire x1="57.912" y1="36.957" x2="57.404" y2="37.465" width="0.508" layer="1"/>
 <contactref element="U$20" pad="RX1"/>
@@
 <signal name="D1">
 <contactref element="U$10" pad="TX"/>
-<wire x1="53.8226" y1="29.1546" x2="43.3106" y2="18.6426" width="0.508" layer="1"/>
-<wire x1="53.8226" y1="29.1546" x2="55.8546" y2="29.1546" width="0.508" layer="1"/>
+<wire x1="53.3146" y1="28.6466" x2="43.3106" y2="18.6426" width="0.508" layer="1"/>
+<wire x1="53.3146" y1="28.6466" x2="56.134" y2="28.6466" width="0.508" layer="1"/>
 <contactref element="U$20" pad="TX0"/>
-<wire x1="55.8546" y1="29.1546" x2="56.134" y2="29.434" width="0.6096" layer="1"/>
 <wire x1="56.134" y1="34.925" x2="56.007" y2="35.052" width="0.6096" layer="1"/>
-<wire x1="56.134" y1="29.434" x2="56.134" y2="34.925" width="0.6096" layer="1"/>
+<wire x1="56.134" y1="28.6466" x2="56.134" y2="34.925" width="0.6096" layer="1"/>
 </signal>
 <signal name="D11">
@@
 <contactref element="IC3" pad="2"/>
 <contactref element="IC4" pad="3"/>
-<wire x1="43.3106" y1="21.1826" x2="43.3106" y2="29.21" width="0.508" layer="1"/>
-<wire x1="44.323" y1="29.21" x2="43.18" y2="30.353" width="0.508" layer="1"/>
-<wire x1="43.18" y1="30.353" x2="43.18" y2="41.402" width="0.508" layer="1"/>
-<wire x1="41.8338" y1="42.7482" x2="43.18" y2="41.402" width="0.508" layer="1"/>
+<wire x1="43.3106" y1="21.1826" x2="43.3106" y2="28.956" width="0.508" layer="1"/>
+<wire x1="43.307" y1="28.702" x2="43.307" y2="41.275" width="0.508" layer="1"/>
+<wire x1="41.8338" y1="42.7482" x2="43.307" y2="41.275" width="0.508" layer="1"/>
 <wire x1="34.4932" y1="52.3494" x2="34.5948" y2="52.2478" width="0.508" layer="1"/>
 <contactref element="R17" pad="2"/>
@@
 <wire x1="31.0388" y1="43.0022" x2="23.4188" y2="43.0022" width="0.6096" layer="1"/>
 <wire x1="40.284" y1="24.638" x2="40.284" y2="27.686" width="0.6096" layer="1"/>
-<wire x1="40.284" y1="27.686" x2="41.808" y2="29.21" width="0.6096" layer="1"/>
-<wire x1="41.808" y1="29.21" x2="43.3106" y2="29.21" width="0.6096" layer="1"/>
+<wire x1="40.284" y1="27.686" x2="41.554" y2="28.956" width="0.6096" layer="1"/>
+<wire x1="41.554" y1="28.956" x2="43.3106" y2="28.956" width="0.6096" layer="1"/>
 <wire x1="31.496" y1="20.168" x2="24.257" y2="20.168" width="0.6096" layer="1"/>
 <wire x1="24.257" y1="20.168" x2="24.13" y2="20.295" width="0.6096" layer="1"/>
