File: LightSwitch-RS485/board.brd (EAGLE design)
At the start: 92.7 x 87.6 mm, 86 parts, among them IC1 PCF8574T, IC2 PCF8574T, K1 OMRON-G3MB-202P-SSR, K2 OMRON-G3MB-202P-SSR, K20 691218410003, K21 691218410003, K22 691218410003, K3 OMRON-G3MB-202P-SSR, K4 OMRON-G3MB-202P-SSR, K5 OMRON-G3MB-202P-SSR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

Commit message: WIP
Parts:
- C5: value (none) -> 100n
- R1, R17, R18, R19: value (none) -> 10k
- R10: value (none) -> 1k
- R20: value (none) -> 120R
Changed lines of the file:
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@@
 <attribute name="VALUE" x="81.026" y="52.832" size="1.27" layer="27" rot="R90"/>
 </element>
-<element name="R10" library="eagle-ltspice" library_urn="urn:adsk.eagle:library:217" package="R1206" package3d_urn="urn:adsk.eagle:package:13301/1" value="" x="69.596" y="45.974" smashed="yes">
+<element name="R10" library="eagle-ltspice" library_urn="urn:adsk.eagle:library:217" package="R1206" package3d_urn="urn:adsk.eagle:package:13301/1" value="1k" x="69.596" y="45.974" smashed="yes">
 <attribute name="NAME" x="70.612" y="43.18" size="1.27" layer="25"/>
 <attribute name="SPICEMODEL" value="NONE" x="69.596" y="45.974" size="1.778" layer="27" display="off"/>
@@
 <attribute name="VALUE" x="14.224" y="-9.779" size="1.27" layer="27" rot="R90"/>
 </element>
-<element name="R1" library="eagle-ltspice" library_urn="urn:adsk.eagle:library:217" package="R1206" package3d_urn="urn:adsk.eagle:package:13301/1" value="" x="2.54" y="-15.24" smashed="yes">
+<element name="R1" library="eagle-ltspice" library_urn="urn:adsk.eagle:library:217" package="R1206" package3d_urn="urn:adsk.eagle:package:13301/1" value="10k" x="2.54" y="-15.24" smashed="yes">
 <attribute name="NAME" x="1.27" y="-13.97" size="1.27" layer="25"/>
 <attribute name="SPICEMODEL" value="NONE" x="2.54" y="-15.24" size="1.778" layer="27" display="off"/>
@@
 <attribute name="VALUE" x="-20.574" y="-45.974" size="0.4064" layer="27"/>
 </element>
-<element name="R17" library="eagle-ltspice" library_urn="urn:adsk.eagle:library:217" package="R1206" package3d_urn="urn:adsk.eagle:package:13301/1" value="" x="-20.32" y="-49.784" smashed="yes">
+<element name="R17" library="eagle-ltspice" library_urn="urn:adsk.eagle:library:217" package="R1206" package3d_urn="urn:adsk.eagle:package:13301/1" value="10k" x="-20.32" y="-49.784" smashed="yes">
 <attribute name="NAME" x="-21.59" y="-48.514" size="1.27" layer="25"/>
 <attribute name="SPICEMODEL" value="NONE" x="-20.32" y="-49.784" size="1.778" layer="27" display="off"/>
@@
 <attribute name="VALUE" x="-21.59" y="-52.324" size="1.27" layer="27"/>
 </element>
-<element name="R18" library="eagle-ltspice" library_urn="urn:adsk.eagle:library:217" package="R1206" package3d_urn="urn:adsk.eagle:package:13301/1" value="" x="-20.32" y="-54.102" smashed="yes">
+<element name="R18" library="eagle-ltspice" library_urn="urn:adsk.eagle:library:217" package="R1206" package3d_urn="urn:adsk.eagle:package:13301/1" value="10k" x="-20.32" y="-54.102" smashed="yes">
 <attribute name="NAME" x="-21.59" y="-52.832" size="1.27" layer="25"/>
 <attribute name="SPICEMODEL" value="NONE" x="-20.32" y="-54.102" size="1.778" layer="27" display="off"/>
@@
 <attribute name="VALUE" x="-22.098" y="-72.39" size="1.27" layer="27"/>
 </element>
-<element name="C5" library="eagle-ltspice" library_urn="urn:adsk.eagle:library:217" package="C0805" package3d_urn="urn:adsk.eagle:package:13265/1" value="" x="-20.828" y="-74.168" smashed="yes">
+<element name="C5" library="eagle-ltspice" library_urn="urn:adsk.eagle:library:217" package="C0805" package3d_urn="urn:adsk.eagle:package:13265/1" value="100n" x="-20.828" y="-74.168" smashed="yes">
 <attribute name="NAME" x="-22.098" y="-72.898" size="1.27" layer="25"/>
 <attribute name="SPICEMODEL" value="NONE" x="-20.828" y="-74.168" size="1.778" layer="27" display="off"/>
@@
 <attribute name="VALUE" x="-22.098" y="-76.708" size="1.27" layer="27"/>
 </element>
-<element name="R19" library="eagle-ltspice" library_urn="urn:adsk.eagle:library:217" package="R1206" package3d_urn="urn:adsk.eagle:package:13301/1" value="" x="-20.32" y="-78.486" smashed="yes">
+<element name="R19" library="eagle-ltspice" library_urn="urn:adsk.eagle:library:217" package="R1206" package3d_urn="urn:adsk.eagle:package:13301/1" value="10k" x="-20.32" y="-78.486" smashed="yes">
 <attribute name="NAME" x="-21.59" y="-77.216" size="1.27" layer="25"/>
 <attribute name="SPICEMODEL" value="NONE" x="-20.32" y="-78.486" size="1.778" layer="27" display="off"/>
@@
 <attribute name="VALUE" x="-21.59" y="-81.026" size="1.27" layer="27"/>
 </element>
-<element name="R20" library="eagle-ltspice" library_urn="urn:adsk.eagle:library:217" package="R1206" package3d_urn="urn:adsk.eagle:package:13301/1" value="" x="-20.32" y="-82.804" smashed="yes">
+<element name="R20" library="eagle-ltspice" library_urn="urn:adsk.eagle:library:217" package="R1206" package3d_urn="urn:adsk.eagle:package:13301/1" value="120R" x="-20.32" y="-82.804" smashed="yes">
 <attribute name="NAME" x="-21.59" y="-81.534" size="1.27" layer="25"/>
 <attribute name="SPICEMODEL" value="NONE" x="-20.32" y="-82.804" size="1.778" layer="27" display="off"/>

Commit message: board
Parts:
- moved K9 314.1 mm to (46.2, 79.5), turned to 180 degrees
- moved ISP1 253.2 mm to (5.84, 35.8), turned to 90 degrees
- moved C13 252.7 mm to (27.9, 29.5), turned to 90 degrees
- moved C12 248.9 mm to (30.5, 29.5), turned to 90 degrees
- moved C11 245.3 mm to (33.0, 29.5), turned to 90 degrees
- moved C10 241.6 mm to (35.6, 29.5), turned to 90 degrees
- moved C9 238.0 mm to (38.1, 29.5), turned to 90 degrees
- moved C8 234.5 mm to (40.6, 29.5), turned to 90 degrees
- moved C7 231.0 mm to (43.2, 29.5), turned to 90 degrees
- moved C6 227.6 mm to (45.7, 29.5), turned to 90 degrees
- moved R37 204.8 mm to (48.0, 9.14), turned to 270 degrees
- moved R36 199.9 mm to (45.5, 9.14), turned to 270 degrees
- moved R35 194.9 mm to (42.9, 9.14), turned to 270 degrees
- moved R34 190.0 mm to (40.4, 9.14), turned to 270 degrees
- moved R33 185.1 mm to (37.8, 9.14), turned to 270 degrees
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Connections:
- net N$51 renamed A
- net N$52 renamed B
- removed net N$18: C3.1, C4.1, C5.1, ISP1.6, U1.5, U2.21, U2.3, U2.5, X1.4
- net GND: now also C3.1, C4.1, C5.1, ISP1.6, U1.5, U2.21, U2.3, U2.5, X1.1
- net VCC: now also X1.4; no longer X1.1
Routing:
- net GND: track 227.4 -> 502.2 mm, vias 8 -> 5
- net VCC: track 212.1 -> 333.9 mm, vias 0 -> 3
- net N$24: track 0.00 -> 68.4 mm, vias 0 -> 2
- net N$23: track 0.00 -> 64.2 mm, vias 0 -> 2
- net N$22: track 0.00 -> 61.1 mm, vias 0 -> 2
- net N$21: track 0.00 -> 55.6 mm, vias 0 -> 2
- net SCL: track 0.00 -> 53.5 mm, vias 0 -> 2
- net SDA: track 0.00 -> 50.5 mm, vias 0 -> 2
- net N$1: track 0.00 -> 47.8 mm, vias 0 -> 2
- net N$15: track 0.00 -> 46.9 mm, vias 0 -> 2
- net N$16: track 0.00 -> 46.1 mm, vias 0 -> 2
- net N$19: track 0.00 -> 44.4 mm, vias 0 -> 2
- net N$26: track 0.00 -> 37.2 mm
- net N$54: track 67.3 -> 30.6 mm
- net N$55: track 3.68 -> 31.2 mm
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- added copper zone on layer 16, net GND
Other:
- board text added: "1 2 L"
- board text added: "3 4 L"
- board text added: "5 6 L"
- board text added: "A B 5V"
- board text added: "GND"
- board text added: "L 8 7"
- board text added: "Light Switch v1.0 falcon.software www.weblogic.pl"
- board text added: "VCC"
- board text removed: "WebLogic DIN Switch v1.0"
