File: LightSwitch-RS485/board.brd (EAGLE design)
At the start: 92.7 x 87.6 mm, 86 parts, among them IC1 PCF8574T, IC2 PCF8574T, K1 OMRON-G3MB-202P-SSR, K2 OMRON-G3MB-202P-SSR, K20 691218410003, K21 691218410003, K22 691218410003, K3 OMRON-G3MB-202P-SSR, K4 OMRON-G3MB-202P-SSR, K5 OMRON-G3MB-202P-SSR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

Commit message: fixes
Parts:
- added T10, T11, T12, T13, T14, T15, T16, T9: BC847, nxp_60:SOT23
- moved R11 62.0 mm to (23.6, 51.8), turned to 270 degrees
- moved R2 49.6 mm to (35.1, 48.5), turned to 90 degrees
- moved R12 22.2 mm to (88.1, 36.6), turned to 270 degrees
- moved R13 20.3 mm to (80.0, 49.8), turned to 270 degrees
- moved R15 19.6 mm to (57.1, 51.6), turned to 270 degrees
- moved R16 19.5 mm to (45.7, 49.0), turned to 270 degrees
- moved R14 19.4 mm to (68.1, 51.1), turned to 270 degrees
- moved R5 5.01 mm to (48.5, 49.0)
- moved R4 4.77 mm to (37.3, 48.5)
- moved R10 4.32 mm to (68.6, 40.9)
- moved R21 4.07 mm to (30.5, 44.7), turned to 90 degrees
- moved R7 3.61 mm to (71.1, 51.1)
- moved R6 3.25 mm to (59.7, 51.6)
- moved R8 3.06 mm to (83.3, 49.8)
- moved R3 2.17 mm to (26.4, 51.6)
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Connections:
- removed net N$2: R1.2, R10.2, T8.1
- new net N$18: R10.2, T16.1
- new net N$51: R12.1, T15.3, T7.1
- new net N$52: R14.1, T13.3, T5.1
- new net N$56: R13.1, T14.3, T6.1
- new net N$67: R5.2, T11.1
- new net N$68: R6.2, T12.1
- new net N$70: R7.2, T13.1
- new net N$73: R8.2, T14.1
- new net N$75: R9.2, T15.1
- net GND: now also T10.2, T11.2, T12.2, T13.2, T14.2, T15.2, T16.2, T9.2; no longer R1.1, R11.1, R12.1, R13.1, R14.1, R15.1, R16.1, R2.1
- net N$5: now also R1.1, T16.3, T8.1; no longer R2.2, R9.2, T7.1
- net N$59: now also R11.1, T9.3; no longer R16.2, R3.2
- net N$61: now also R2.2, T10.3; no longer R15.2, R4.2
- net N$63: now also R3.2, T9.1; no longer R14.2, R5.2, T1.1
- net N$64: now also R4.2, T10.1; no longer R13.2, R6.2, T4.1
- net N$65: now also R16.1, T1.1, T11.3; no longer R12.2, R7.2, T5.1
- net N$66: now also R15.1, T12.3, T4.1; no longer R11.2, R8.2, T6.1
- net VCC: now also R1.2, R11.2, R12.2, R13.2, R14.2, R15.2, R16.2, R2.1
Routing:
- net VCC: track 333.9 -> 424.3 mm
- net GND: track 502.2 -> 459.8 mm
- net N$18: track 0.00 -> 9.30 mm
- net N$2: track 7.06 -> 0.00 mm
- net N$56: track 0.00 -> 6.82 mm
- net N$52: track 0.00 -> 6.58 mm
- net N$4: track 34.1 -> 27.9 mm
- net N$51: track 0.00 -> 5.63 mm
- net N$6: track 25.1 -> 19.8 mm
- net N$64: track 9.10 -> 4.01 mm
- net N$11: track 16.4 -> 12.1 mm
- net N$63: track 6.27 -> 2.23 mm
- net N$3: track 41.3 -> 37.5 mm
- net N$67: track 0.00 -> 2.88 mm
- net N$75: track 0.00 -> 2.64 mm
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Other:
- board text added: "Light Switch v2.0 falcon.software www.weblogic.pl"
- board text removed: "Light Switch v1.0 falcon.software www.weblogic.pl"
