File: LightSwitch-RS485/board.sch (EAGLE design)
At the start: 86 parts, among them IC1 PCF8574T, IC2 PCF8574T, K1 OMRON-G3MB-202P-SSR, K2 OMRON-G3MB-202P-SSR, K20 691218410003, K21 691218410003, K22 691218410003, K3 OMRON-G3MB-202P-SSR, K4 OMRON-G3MB-202P-SSR, K5 OMRON-G3MB-202P-SSR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

Commit message: WIP
Parts:
- C5: value (none) -> 100n
- R1, R17, R18, R19: value (none) -> 10k
- R10: value (none) -> 1k
- R20: value (none) -> 120R
Changed lines of the file:
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@@
 <part name="R8" library="eagle-ltspice" library_urn="urn:adsk.eagle:library:217" deviceset="R" device="R1206" package3d_urn="urn:adsk.eagle:package:13301/1"/>
 <part name="R9" library="eagle-ltspice" library_urn="urn:adsk.eagle:library:217" deviceset="R" device="R1206" package3d_urn="urn:adsk.eagle:package:13301/1"/>
-<part name="R10" library="eagle-ltspice" library_urn="urn:adsk.eagle:library:217" deviceset="R" device="R1206" package3d_urn="urn:adsk.eagle:package:13301/1"/>
+<part name="R10" library="eagle-ltspice" library_urn="urn:adsk.eagle:library:217" deviceset="R" device="R1206" package3d_urn="urn:adsk.eagle:package:13301/1" value="1k"/>
 <part name="T1" library="transistor" library_urn="urn:adsk.eagle:library:402" deviceset="BC847" device="" package3d_urn="urn:adsk.eagle:package:29904/2"/>
 <part name="T2" library="transistor" library_urn="urn:adsk.eagle:library:402" deviceset="BC847" device="" package3d_urn="urn:adsk.eagle:package:29904/2"/>
@@
 <part name="T8" library="transistor" library_urn="urn:adsk.eagle:library:402" deviceset="BC847" device="" package3d_urn="urn:adsk.eagle:package:29904/2"/>
 <part name="IC1" library="micro-philips" library_urn="urn:adsk.eagle:library:290" deviceset="PCF8574" device="T" package3d_urn="urn:adsk.eagle:package:20172/1"/>
-<part name="R1" library="eagle-ltspice" library_urn="urn:adsk.eagle:library:217" deviceset="R" device="R1206" package3d_urn="urn:adsk.eagle:package:13301/1"/>
+<part name="R1" library="eagle-ltspice" library_urn="urn:adsk.eagle:library:217" deviceset="R" device="R1206" package3d_urn="urn:adsk.eagle:package:13301/1" value="10k"/>
 <part name="R2" library="eagle-ltspice" library_urn="urn:adsk.eagle:library:217" deviceset="R" device="R1206" package3d_urn="urn:adsk.eagle:package:13301/1"/>
 <part name="R11" library="eagle-ltspice" library_urn="urn:adsk.eagle:library:217" deviceset="R" device="R1206" package3d_urn="urn:adsk.eagle:package:13301/1"/>
@@
 <part name="U1" library="MAX487ESA_TCBX" deviceset="MAX487ESA+TCBX" device=""/>
 <part name="U2" library="thecustomgeek" deviceset="ATMEGA328" device=""/>
-<part name="R17" library="eagle-ltspice" library_urn="urn:adsk.eagle:library:217" deviceset="R" device="R1206" package3d_urn="urn:adsk.eagle:package:13301/1"/>
-<part name="R18" library="eagle-ltspice" library_urn="urn:adsk.eagle:library:217" deviceset="R" device="R1206" package3d_urn="urn:adsk.eagle:package:13301/1"/>
+<part name="R17" library="eagle-ltspice" library_urn="urn:adsk.eagle:library:217" deviceset="R" device="R1206" package3d_urn="urn:adsk.eagle:package:13301/1" value="10k"/>
+<part name="R18" library="eagle-ltspice" library_urn="urn:adsk.eagle:library:217" deviceset="R" device="R1206" package3d_urn="urn:adsk.eagle:package:13301/1" value="10k"/>
 <part name="Q1" library="crystal" library_urn="urn:adsk.eagle:library:204" deviceset="CRYSTAL" device="HC49S" package3d_urn="urn:adsk.eagle:package:12071/1"/>
 <part name="C3" library="eagle-ltspice" library_urn="urn:adsk.eagle:library:217" deviceset="C" device="" package3d_urn="urn:adsk.eagle:package:13265/1"/>
 <part name="C4" library="eagle-ltspice" library_urn="urn:adsk.eagle:library:217" deviceset="C" device="" package3d_urn="urn:adsk.eagle:package:13265/1"/>
-<part name="C5" library="eagle-ltspice" library_urn="urn:adsk.eagle:library:217" deviceset="C" device="" package3d_urn="urn:adsk.eagle:package:13265/1"/>
-<part name="R19" library="eagle-ltspice" library_urn="urn:adsk.eagle:library:217" deviceset="R" device="R1206" package3d_urn="urn:adsk.eagle:package:13301/1"/>
-<part name="R20" library="eagle-ltspice" library_urn="urn:adsk.eagle:library:217" deviceset="R" device="R1206" package3d_urn="urn:adsk.eagle:package:13301/1"/>
+<part name="C5" library="eagle-ltspice" library_urn="urn:adsk.eagle:library:217" deviceset="C" device="" package3d_urn="urn:adsk.eagle:package:13265/1" value="100n"/>
+<part name="R19" library="eagle-ltspice" library_urn="urn:adsk.eagle:library:217" deviceset="R" device="R1206" package3d_urn="urn:adsk.eagle:package:13301/1" value="10k"/>
+<part name="R20" library="eagle-ltspice" library_urn="urn:adsk.eagle:library:217" deviceset="R" device="R1206" package3d_urn="urn:adsk.eagle:package:13301/1" value="120R"/>
 <part name="X1" library="Rembrandt Electronics - JST XH Connectors v1-0" deviceset="JST-XH-04-PIN" device="-LONG-PAD"/>
 <part name="X2" library="Rembrandt Electronics - JST XH Connectors v1-0" deviceset="JST-XH-09-PIN" device="-LONG-PAD"/>

Commit message: board
Connections:
- net N$51 renamed A
- net N$52 renamed B
- removed net N$18: C3.1, C4.1, C5.1, ISP1.GND, U1.GND, U2.AGND, U2.GND@1, U2.GND@2, X1-4.S
- net GND: now also C3.1, C4.1, C5.1, ISP1.GND, U1.GND, U2.AGND, U2.GND@1, U2.GND@2, X1-1.S
- net VCC: now also X1-4.S; no longer X1-1.S
Other:
- moved on the sheet: X1-1, X1-4

Commit message: fixes
Parts:
- added T10, T11, T12, T13, T14, T15, T16, T9: BC847, nxp_60:BC847
Connections:
- removed net N$2: R1.2, R10.2, T8.B
- new net N$18: R10.2, T16.B
- new net N$51: R12.1, T15.C, T7.B
- new net N$52: R14.1, T13.C, T5.B
- new net N$56: R13.1, T14.C, T6.B
- new net N$67: R5.2, T11.B
- new net N$68: R6.2, T12.B
- new net N$70: R7.2, T13.B
- new net N$73: R8.2, T14.B
- new net N$75: R9.2, T15.B
- net GND: now also T10.E, T11.E, T12.E, T13.E, T14.E, T15.E, T16.E, T9.E; no longer R1.1, R11.1, R12.1, R13.1, R14.1, R15.1, R16.1, R2.1
- net N$5: now also R1.1, T16.C, T8.B; no longer R2.2, R9.2, T7.B
- net N$59: now also R11.1, T9.C; no longer R16.2, R3.2
- net N$61: now also R2.2, T10.C; no longer R15.2, R4.2
- net N$63: now also R3.2, T9.B; no longer R14.2, R5.2, T1.B
- net N$64: now also R4.2, T10.B; no longer R13.2, R6.2, T4.B
- net N$65: now also R16.1, T1.B, T11.C; no longer R12.2, R7.2, T5.B
- net N$66: now also R15.1, T12.C, T4.B; no longer R11.2, R8.2, T6.B
- net VCC: now also R1.2, R11.2, R12.2, R13.2, R14.2, R15.2, R16.2, R2.1
Other:
- moved on the sheet: IC1, R1, R10, R11, R12, R13, R14, R15, R16, R2, R3, R4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
